Commit message: Gazebo Map created

File: sr_description/urdf/wall.urdf.xacro (robot description, xacro)
@@ -45,5 +45,5 @@
       <child link="back_wall"/>
       <!-- Back of chassis, on top -->
-      <origin xyz="${-0.2} ${wall_length/2} ${0.12}" rpy="0 0 0"/>
+      <origin xyz="${-0.2} ${wall_length/2} ${0.045}" rpy="0 0 0"/>
     </joint>
   </xacro:macro>
