Commit message: visualised bot

File: sr_description/urdf/base.urdf.xacro (robot description, xacro)
@@ -1,60 +1,31 @@
 <?xml version="1.0"?>
-<robot xmlns:xacro="http://www.ros.org/wiki/xacro" name="base">
-  <!-- ========================================
-       BASE CHASSIS - SQUARE 40x40x20 cm
-       ======================================== -->
-  <!-- Robot parameters -->
-  <xacro:property name="chassis_length" value="0.40"/>
-  <xacro:property name="chassis_width" value="0.40"/>
-  <xacro:property name="chassis_height" value="0.20"/>
-  <xacro:property name="chassis_mass" value="5.0"/>
-  <!-- Wheel mounting positions -->
-  <xacro:property name="wheel_x_offset" value="0.17"/>
-  <xacro:property name="wheel_y_offset" value="0.17"/>
-  <xacro:property name="wheel_z_height" value="0.05"/>
+<robot xmlns:xacro="http://www.ros.org/wiki/xacro">
   <xacro:macro name="create_base">
-    <!-- BASE LINK (MAIN CHASSIS) -->
     <link name="base_link">
-      <inertial>
-        <origin xyz="0 0 0" rpy="0 0 0"/>
-        <mass value="${chassis_mass}"/>
-        <!-- Inertia for rectangular box -->
-        <inertia
-          ixx="${chassis_mass * (chassis_width*chassis_width + chassis_height*chassis_height) / 12.0}"
-          iyy="${chassis_mass * (chassis_length*chassis_length + chassis_height*chassis_height) / 12.0}"
-          izz="${chassis_mass * (chassis_length*chassis_length + chassis_width*chassis_width) / 12.0}"
-          ixy="0" ixz="0" iyz="0"/>
-      </inertial>
-      <!-- Visual: Simple grey box (40x40x20 cm) -->
       <visual>
-        <origin xyz="0 0 ${chassis_height/2}" rpy="0 0 0"/>
+        <origin xyz="0 0 0.1"/>
         <geometry>
-          <box size="${chassis_length} ${chassis_width} ${chassis_height}"/>
+          <box size="0.44 0.4 0.1"/>
         </geometry>
         <material name="grey"/>
       </visual>
-      <!-- Collision: Same box shape -->
       <collision>
-        <origin xyz="0 0 ${chassis_height/2}" rpy="0 0 0"/>
+        <origin xyz="0 0 0.1"/>
         <geometry>
-          <box size="${chassis_length} ${chassis_width} ${chassis_height}"/>
+          <box size="0.44 0.4 0.1"/>
         </geometry>
       </collision>
-    </link>
-    <!-- ARM MOUNTING POINT (for future arm attachment) -->
-    <!-- This is where the arm will be attached -->
-    <link name="arm_base">
       <inertial>
-        <origin xyz="0 0 0" rpy="0 0 0"/>
-        <mass value="0.01"/>
-        <inertia ixx="0.001" iyy="0.001" izz="0.001" ixy="0" ixz="0" iyz="0"/>
+        <mass value="5.0"/>
+        <inertia ixx="0.1" iyy="0.1" izz="0.1"
+                 ixy="0" ixz="0" iyz="0"/>
       </inertial>
     </link>
-    <!-- ARM BASE JOINT (fixed to top of chassis) -->
-    <joint name="arm_base_joint" type="fixed">
+    <!-- arm mount -->
+    <link name="arm_base_link"/>
+    <joint name="arm_mount_joint" type="fixed">
       <parent link="base_link"/>
-      <child link="arm_base"/>
-      <!-- Positioned at top center of chassis -->
-      <origin xyz="0 0 ${chassis_height}" rpy="0 0 0"/>
+      <child link="arm_base_link"/>
+      <origin xyz="0.16 0 0.15"/>
     </joint>
   </xacro:macro>

File: sr_description/urdf/gazebo.urdf.xacro (robot description, xacro)
@@ -1,61 +1,79 @@
 <?xml version="1.0"?>
-<robot xmlns:xacro="http://www.ros.org/wiki/xacro" name="gazebo_setup">
-  <!-- ========================================
-       GAZEBO SPECIFIC SETUP
-       NO VISUAL/COLLISION HERE - DEBUGGING FRIENDLY
-       ======================================== -->
+<robot xmlns:xacro="http://www.ros.org/wiki/xacro">
   <xacro:macro name="gazebo_setup">
-    <!-- Differential Drive Plugin -->
-    <gazebo>
-      <plugin name="differential_drive_controller" filename="libgazebo_ros_diff_drive.so">
-        <!-- Wheel joints -->
-        <left_joint>wheel_fl_joint</left_joint>
-        <right_joint>wheel_fr_joint</right_joint>
-        <!-- Kinematics -->
-        <wheel_separation>0.40</wheel_separation>
-        <wheel_diameter>0.10</wheel_diameter>
-        <!-- Limits -->
-        <max_wheel_torque>20</max_wheel_torque>
-        <max_wheel_acceleration>10</max_wheel_acceleration>
-        <!-- Frames -->
-        <odometry_frame>odom</odometry_frame>
-        <robot_base_frame>base_link</robot_base_frame>
-        <!-- ROS interface -->
-        <ros>
-          <remapping>cmd_vel:=cmd_vel</remapping>
-          <remapping>odom:=odom</remapping>
-        </ros>
-        <!-- Output -->
-        <publish_odom>true</publish_odom>
-        <publish_odom_tf>true</publish_odom_tf>
-        <publish_wheel_tf>true</publish_wheel_tf>
-      </plugin>
-    </gazebo>
-    <!-- Base link material -->
+    <!-- ================= BASE ================= -->
     <gazebo reference="base_link">
       <material>Gazebo/Grey</material>
-      <mu1>0.2</mu1>
-      <mu2>0.2</mu2>
+      <mu1>0.3</mu1>
+      <mu2>0.3</mu2>
     </gazebo>
-    <!-- Wheel materials and friction -->
+    <!-- ================= MECANUM WHEELS ================= -->
     <gazebo reference="wheel_fl">
-      <mu1>1.5</mu1>
-      <mu2>1.5</mu2>
+      <mu1>2.0</mu1>
+      <mu2>2.0</mu2>
       <material>Gazebo/Black</material>
     </gazebo>
     <gazebo reference="wheel_fr">
-      <mu1>1.5</mu1>
-      <mu2>1.5</mu2>
+      <mu1>2.0</mu1>
+      <mu2>2.0</mu2>
       <material>Gazebo/Black</material>
     </gazebo>
     <gazebo reference="wheel_bl">
-      <mu1>1.5</mu1>
-      <mu2>1.5</mu2>
+      <mu1>2.0</mu1>
+      <mu2>2.0</mu2>
       <material>Gazebo/Black</material>
     </gazebo>
     <gazebo reference="wheel_br">
-      <mu1>1.5</mu1>
-      <mu2>1.5</mu2>
+      <mu1>2.0</mu2>
+      <mu2>2.0</mu2>
       <material>Gazebo/Black</material>
+    </gazebo>
+    <!-- ================= ARM LINKS ================= -->
+    <gazebo reference="arm_base_link">
+      <material>Gazebo/Blue</material>
+      <mu1>0.5</mu1>
+      <mu2>0.5</mu2>
+    </gazebo>
+    <gazebo reference="arm_shoulder_link">
+      <material>Gazebo/Orange</material>
+      <mu1>0.5</mu1>
+      <mu2>0.5</mu2>
+    </gazebo>
+    <gazebo reference="arm_elbow_link">
+      <material>Gazebo/Orange</material>
+      <mu1>0.5</mu1>
+      <mu2>0.5</mu2>
+    </gazebo>
+    <gazebo reference="arm_wrist_link">
+      <material>Gazebo/Yellow</material>
+      <mu1>0.4</mu1>
+      <mu2>0.4</mu2>
+    </gazebo>
+    <gazebo reference="gripper_link">
+      <material>Gazebo/Red</material>
+      <mu1>0.8</mu1>
+      <mu2>0.8</mu2>
+    </gazebo>
+    <!-- ================= ARM JOINT DYNAMICS ================= -->
+    <gazebo reference="shoulder_joint">
+      <provideFeedback>true</provideFeedback>
+      <implicitSpringDamper>true</implicitSpringDamper>
+    </gazebo>
+    <gazebo reference="elbow_joint">
+      <provideFeedback>true</provideFeedback>
+      <implicitSpringDamper>true</implicitSpringDamper>
+    </gazebo>
+    <gazebo reference="wrist_joint">
+      <provideFeedback>true</provideFeedback>
+      <implicitSpringDamper>true</implicitSpringDamper>
+    </gazebo>
+    <!-- ================= BASIC ODOM (TEMP DEBUG) ================= -->
+    <gazebo>
+      <plugin name="odom_plugin" filename="libgazebo_ros_p3d.so">
+        <bodyName>base_link</bodyName>
+        <topicName>odom</topicName>
+        <frameName>odom</frameName>
+        <updateRate>50.0</updateRate>
+      </plugin>
     </gazebo>
   </xacro:macro>

File: sr_description/urdf/robot.urdf.xacro (robot description, xacro)
@@ -1,16 +1,10 @@
 <?xml version="1.0"?>
-<robot xmlns:xacro="http://www.ros.org/wiki/xacro" name="square_mecanum_robot">
-  <!-- ========================================
-       MAIN ROBOT FILE - INCLUDES ALL PARTS
-       ======================================== -->
-  <!-- Include all xacro files -->
-  <xacro:include filename="$(find sr_description)/urdf/materials.urdf.xacro"/>
+<robot xmlns:xacro="http://www.ros.org/wiki/xacro" name="lifter_bot">
+  <xacro:include filename="$(find sr_description)/urdf/material.urdf.xacro"/>
   <xacro:include filename="$(find sr_description)/urdf/base.urdf.xacro"/>
-  <xacro:include filename="$(find sr_description)/urdf/wheels.urdf.xacro"/>
-  <xacro:include filename="$(find sr_description)/urdf/gazebo.urdf.xacro"/>
-  <!-- Create the robot -->
+  <xacro:include filename="$(find sr_description)/urdf/wheel.urdf.xacro"/>
+  <xacro:include filename="$(find sr_description)/urdf/arm.urdf.xacro"/>
   <xacro:create_base/>
   <xacro:create_wheels/>
-  <!-- Gazebo setup (separate from visual/collision) -->
-  <xacro:gazebo_setup/>
+  <xacro:create_arm/>
 </robot>

File: sr_description/urdf/wheel.urdf.xacro (robot description, xacro)
@@ -1,61 +1,37 @@
 <?xml version="1.0"?>
-<robot xmlns:xacro="http://www.ros.org/wiki/xacro" name="wheels">
-  <!-- ========================================
-       MECANUM WHEELS - STL MESHES
-       ======================================== -->
-  <!-- Wheel parameters -->
-  <xacro:property name="wheel_radius" value="0.05"/>
-  <xacro:property name="wheel_width" value="0.04"/>
-  <xacro:property name="wheel_mass" value="0.5"/>
-  <!-- Mesh paths -->
-  <xacro:property name="mesh_path" value="package://sr_description/meshes/"/>
-  <!-- Mecanum wheel macro -->
-  <xacro:macro name="mecanum_wheel" params="wheel_name wheel_type pos_x pos_y">
-    <link name="${wheel_name}">
-      <inertial>
-        <origin xyz="0 0 0" rpy="0 0 0"/>
-        <mass value="${wheel_mass}"/>
-        <inertia
-          ixx="${wheel_mass * wheel_radius * wheel_radius / 4}"
-          iyy="${wheel_mass * (wheel_radius*wheel_radius + wheel_width*wheel_width) / 12}"
-          izz="${wheel_mass * wheel_radius * wheel_radius / 4}"
-          ixy="0" ixz="0" iyz="0"/>
-      </inertial>
-      <!-- Visual: STL mesh for mecanum wheel -->
+<robot xmlns:xacro="http://www.ros.org/wiki/xacro">
+  <xacro:macro name="mecanum_wheel" params="name x y mesh">
+    <link name="${name}">
       <visual>
-        <origin xyz="0 0 0" rpy="1.5708 0 0"/>
+        <origin rpy="0 0 0"/>
         <geometry>
-          <mesh filename="${mesh_path}mecanum_wheel_${wheel_type}.stl" scale="1.0 1.0 1.0"/>
+          <mesh filename="package://sr_description/meshes/${mesh}" scale="0.0018  0.0018 0.0018 "/>
         </geometry>
         <material name="dark_grey"/>
       </visual>
-      <!-- Collision: Simple cylinder (fast physics) -->
       <collision>
-        <origin xyz="0 0 0" rpy="1.5708 0 0"/>
+        <origin rpy="0 0 0"/>
         <geometry>
-          <cylinder radius="${wheel_radius}" length="${wheel_width}"/>
+          <cylinder radius="0.05" length="0.04"/>
         </geometry>
       </collision>
+      <inertial>
+        <mass value="0.5"/>
+        <inertia ixx="0.001" iyy="0.001" izz="0.001"
+                 ixy="0" ixz="0" iyz="0"/>
+      </inertial>
     </link>
-    <!-- Wheel joint -->
-    <joint name="${wheel_name}_joint" type="continuous">
+    <joint name="${name}_joint" type="continuous">
       <parent link="base_link"/>
-      <child link="${wheel_name}"/>
-      <origin xyz="${pos_x} ${pos_y} 0.05" rpy="0 0 0"/>
+      <child link="${name}"/>
+      <origin xyz="${x} ${y} 0.05"/>
       <axis xyz="0 1 0"/>
-      <limit effort="20" velocity="10"/>
-      <dynamics damping="0.01" friction="0.01"/>
     </joint>
   </xacro:macro>
-  <!-- Create all 4 wheels -->
   <xacro:macro name="create_wheels">
-    <!-- Front-Left (LEFT type) -->
-    <xacro:mecanum_wheel wheel_name="wheel_fl" wheel_type="left" pos_x="0.17" pos_y="0.17"/>
-    <!-- Front-Right (RIGHT type) -->
-    <xacro:mecanum_wheel wheel_name="wheel_fr" wheel_type="right" pos_x="0.17" pos_y="-0.17"/>
-    <!-- Back-Left (RIGHT type - diagonal opposite) -->
-    <xacro:mecanum_wheel wheel_name="wheel_bl" wheel_type="right" pos_x="-0.17" pos_y="0.17"/>
-    <!-- Back-Right (LEFT type - diagonal opposite) -->
-    <xacro:mecanum_wheel wheel_name="wheel_br" wheel_type="left" pos_x="-0.17" pos_y="-0.17"/>
+    <xacro:mecanum_wheel name="wheel_fl" x="0.2" y="0.2" mesh="mecanum_wheel_left.STL"/>
+    <xacro:mecanum_wheel name="wheel_fr" x="0.2" y="-0.2" mesh="mecanum_wheel_right.STL"/>
+    <xacro:mecanum_wheel name="wheel_bl" x="-0.2" y="0.2" mesh="mecanum_wheel_right.STL"/>
+    <xacro:mecanum_wheel name="wheel_br" x="-0.2" y="-0.2" mesh="mecanum_wheel_left.STL"/>
   </xacro:macro>
 </robot>

Commit message: building runner bot

File: sr_description/urdf/base.urdf.xacro (robot description, xacro)
@@ -6,5 +6,5 @@
         <origin xyz="0 0 0.1"/>
         <geometry>
-          <box size="0.44 0.4 0.1"/>
+          <box size="0.44 0.31 0.1"/>
         </geometry>
         <material name="grey"/>
@@ -13,5 +13,5 @@
         <origin xyz="0 0 0.1"/>
         <geometry>
-          <box size="0.44 0.4 0.1"/>
+          <box size="0.44 0.31 0.1"/>
         </geometry>
       </collision>

Commit message: urdf draft-3

File: sr_description/urdf/base.urdf.xacro (robot description, xacro)
@@ -2,30 +2,97 @@
 <robot xmlns:xacro="http://www.ros.org/wiki/xacro">
   <xacro:macro name="create_base">
+    <!-- Ground reference frame -->
+    <link name="base_footprint"/>
+    <!-- Actual robot body -->
     <link name="base_link">
       <visual>
-        <origin xyz="0 0 0.1"/>
+        <origin xyz="0 0 0"/>
         <geometry>
-          <box size="0.44 0.31 0.1"/>
+          <box size="0.44 0.36 0.1"/>
         </geometry>
         <material name="grey"/>
       </visual>
       <collision>
-        <origin xyz="0 0 0.1"/>
+        <origin xyz="0 0 0"/>
         <geometry>
-          <box size="0.44 0.31 0.1"/>
+          <box size="0.44 0.36 0.1"/>
         </geometry>
       </collision>
       <inertial>
+        <origin xyz="0 0 0"/>
         <mass value="5.0"/>
         <inertia ixx="0.1" iyy="0.1" izz="0.1"
-                 ixy="0" ixz="0" iyz="0"/>
+                ixy="0" ixz="0" iyz="0"/>
       </inertial>
     </link>
-    <!-- arm mount -->
+    <!-- base_link sits above ground -->
+    <joint name="base_footprint_to_base_link" type="fixed">
+      <parent link="base_footprint"/>
+      <child link="base_link"/>
+      <origin xyz="0 0 0.05"/>
+    </joint>
+    <!-- ================= SHAFT LINKS ================= -->
+    <!-- Shaft FL -->
+    <link name="shaft_fl">
+      <visual>
+        <geometry>
+          <mesh filename="package://sr_description/meshes/wheel_shaft.stl"
+                scale="0.002 0.002 0.002"/>
+        </geometry>
+      </visual>
+    </link>
+    <joint name="shaft_fl_joint" type="fixed">
+      <parent link="base_link"/>
+      <child link="shaft_fl"/>
+      <origin xyz="0.20 0.18 0.0"/>
+    </joint>
+    <!-- Shaft FR -->
+    <link name="shaft_fr">
+      <visual>
+        <geometry>
+          <mesh filename="package://sr_description/meshes/wheel_shaft.stl"
+                scale="0.002 0.002 0.002"/>
+        </geometry>
+      </visual>
+    </link>
+    <joint name="shaft_fr_joint" type="fixed">
+      <parent link="base_link"/>
+      <child link="shaft_fr"/>
+      <origin xyz="0.20 -0.18 0.0" rpy="0 0 3.1416"/>
+    </joint>
+    <!-- Shaft BL -->
+    <link name="shaft_bl">
+      <visual>
+        <geometry>
+          <mesh filename="package://sr_description/meshes/wheel_shaft.stl"
+                scale="0.002 0.002 0.002"/>
+        </geometry>
+      </visual>
+    </link>
+    <joint name="shaft_bl_joint" type="fixed">
+      <parent link="base_link"/>
+      <child link="shaft_bl"/>
+      <origin xyz="-0.20 0.18 0.0"/>
+    </joint>
+    <!-- Shaft BR -->
+    <link name="shaft_br">
+      <visual>
+        <geometry>
+          <mesh filename="package://sr_description/meshes/wheel_shaft.stl"
+                scale="0.002 0.002 0.002"/>
+        </geometry>
+      </visual>
+    </link>
+    <joint name="shaft_br_joint" type="fixed">
+      <parent link="base_link"/>
+      <child link="shaft_br"/>
+      <origin xyz="-0.20 -0.18 0.0" rpy="0 0 3.1416"/>
+    </joint>
+    <!-- ================= ARM MOUNT ================= -->
     <link name="arm_base_link"/>
     <joint name="arm_mount_joint" type="fixed">
       <parent link="base_link"/>
       <child link="arm_base_link"/>
-      <origin xyz="0.16 0 0.15"/>
+      <origin xyz="0.16 0 0.06"/>
     </joint>
   </xacro:macro>

File: sr_description/urdf/wheel.urdf.xacro (robot description, xacro)
@@ -1,5 +1,5 @@
 <?xml version="1.0"?>
 <robot xmlns:xacro="http://www.ros.org/wiki/xacro">
-  <xacro:macro name="mecanum_wheel" params="name x y mesh">
+  <xacro:macro name="mecanum_wheel" params="name x y mesh shaft_link offset">
     <link name="${name}">
       <visual>
@@ -17,4 +17,5 @@
       </collision>
       <inertial>
+        <origin rpy="0 0 0"/>
         <mass value="0.5"/>
         <inertia ixx="0.001" iyy="0.001" izz="0.001"
@@ -23,15 +24,15 @@
     </link>
     <joint name="${name}_joint" type="continuous">
-      <parent link="base_link"/>
+      <parent link="${shaft_link}"/>
       <child link="${name}"/>
-      <origin xyz="${x} ${y} 0.05"/>
+      <origin xyz=" 0 ${offset} 0 "/>
       <axis xyz="0 1 0"/>
     </joint>
   </xacro:macro>
   <xacro:macro name="create_wheels">
-    <xacro:mecanum_wheel name="wheel_fl" x="0.2" y="0.2" mesh="mecanum_wheel_left.stl"/>
-    <xacro:mecanum_wheel name="wheel_fr" x="0.2" y="-0.2" mesh="mecanum_wheel_right.stl"/>
-    <xacro:mecanum_wheel name="wheel_bl" x="-0.2" y="0.2" mesh="mecanum_wheel_right.stl"/>
-    <xacro:mecanum_wheel name="wheel_br" x="-0.2" y="-0.2" mesh="mecanum_wheel_left.stl"/>
+    <xacro:mecanum_wheel name="wheel_fl" x="0.2" y="0.2" mesh="mecanum_wheel_left.stl" shaft_link="shaft_fl" offset= "0.05"/>
+    <xacro:mecanum_wheel name="wheel_fr" x="0.2" y="-0.2" mesh="mecanum_wheel_right.stl" shaft_link="shaft_fr" offset= "0.05"/>
+    <xacro:mecanum_wheel name="wheel_bl" x="-0.2" y="0.2" mesh="mecanum_wheel_right.stl" shaft_link="shaft_bl" offset= "0.05"/>
+    <xacro:mecanum_wheel name="wheel_br" x="-0.2" y="-0.2" mesh="mecanum_wheel_left.stl" shaft_link="shaft_br" offset= "0.05"/>
   </xacro:macro>
 </robot>
