Commit message: complete launch

File: sr_description/urdf/base.urdf.xacro (robot description, xacro)
@@ -21,5 +21,5 @@
       <inertial>
         <origin xyz="0 0 0"/>
-        <mass value="5.0"/>
+        <mass value="1.0"/>
         <inertia ixx="0.1" iyy="0.1" izz="0.1"
                 ixy="0" ixz="0" iyz="0"/>

File: sr_description/urdf/lifter_bot.urdf.xacro (robot description, xacro)
@@ -1,4 +1,5 @@
 <?xml version="1.0"?>
 <robot xmlns:xacro="http://www.ros.org/wiki/xacro" name="lifter_bot">
+  <xacro:arg name="namespace" default=""/>
   <xacro:include filename="$(find sr_description)/urdf/material.urdf.xacro"/>
   <xacro:include filename="$(find sr_description)/urdf/base.urdf.xacro"/>

File: sr_description/urdf/lifter_gazebo.urdf.xacro (robot description, xacro)
@@ -4,23 +4,43 @@
     <!-- ================= BASE ================= -->
     <gazebo reference="base_link">
-      <mu1>0.3</mu1>
-      <mu2>0.3</mu2>
+      <mu1>0</mu1>
+      <mu2>0</mu2>
     </gazebo>
     <!-- ================= MECANUM WHEELS ================= -->
     <gazebo reference="wheel_fl">
-      <mu1>2.0</mu1>
-      <mu2>2.0</mu2>
+        <mu1>10.0</mu1>
+        <mu2>10.0</mu2>
+        <kp>100000.0</kp>
+        <kd>10.0</kd>
+        <minDepth>0.001</minDepth>
+        <maxVel>0.1</maxVel>
+        <fdir1>1 1 0</fdir1>
     </gazebo>
     <gazebo reference="wheel_fr">
-      <mu1>2.0</mu1>
-      <mu2>2.0</mu2>
+        <mu1>10.0</mu1>
+        <mu2>10.0</mu2>
+        <kp>100000.0</kp>
+        <kd>10.0</kd>
+        <minDepth>0.001</minDepth>
+        <maxVel>0.1</maxVel>
+        <fdir1>1 -1 0</fdir1>
     </gazebo>
     <gazebo reference="wheel_bl">
-      <mu1>2.0</mu1>
-      <mu2>2.0</mu2>
+        <mu1>10.0</mu1>
+        <mu2>10.0</mu2>
+        <kp>100000.0</kp>
+        <kd>10.0</kd>
+        <minDepth>0.001</minDepth>
+        <maxVel>0.1</maxVel>
+        <fdir1>1 -1 0</fdir1>
     </gazebo>
     <gazebo reference="wheel_br">
-      <mu1>2.0</mu1>
-      <mu2>2.0</mu2>
+        <mu1>10.0</mu1>
+        <mu2>10.0</mu2>
+        <kp>100000.0</kp>
+        <kd>10.0</kd>
+        <minDepth>0.001</minDepth>
+        <maxVel>0.1</maxVel>
+        <fdir1>1 1 0</fdir1>
     </gazebo>
     <!-- ================= ARM LINKS ================= -->
@@ -42,7 +62,10 @@
     <!-- ================= ROS2 CONTROL (REQUIRED) ================= -->
     <gazebo>
-        <plugin filename="ign_ros2_control-system" name="ign_ros2_control::IgnitionROS2ControlPlugin">
-            <parameters>$(find sr_control)/config/lifter_config.yaml</parameters>
-        </plugin>
+      <plugin filename="ign_ros2_control-system" name="ign_ros2_control::IgnitionROS2ControlPlugin">
+        <ros>
+          <namespace>$(arg namespace)</namespace>
+        </ros>
+        <parameters>$(find sr_control)/config/lifter_config.yaml</parameters>
+      </plugin>
     </gazebo>
   </xacro:macro>

File: sr_description/urdf/runner_bot.urdf.xacro (robot description, xacro)
@@ -1,4 +1,5 @@
 <?xml version="1.0"?>
 <robot xmlns:xacro="http://www.ros.org/wiki/xacro" name="runner_bot">
+  <xacro:arg name="namespace" default=""/>
   <xacro:include filename="$(find sr_description)/urdf/material.urdf.xacro"/>
   <xacro:include filename="$(find sr_description)/urdf/base.urdf.xacro"/>

File: sr_description/urdf/runner_gazebo.urdf.xacro (robot description, xacro)
@@ -9,18 +9,38 @@
     <!-- ================= MECANUM WHEELS ================= -->
     <gazebo reference="wheel_fl">
-      <mu1>2.0</mu1>
-      <mu2>2.0</mu2>
+        <mu1>1.0</mu1>
+        <mu2>1.0</mu2>
+        <kp>100000.0</kp>
+        <kd>10.0</kd>
+        <minDepth>0.001</minDepth>
+        <maxVel>0.1</maxVel>
+        <fdir1>1 0 0</fdir1>
     </gazebo>
     <gazebo reference="wheel_fr">
-      <mu1>2.0</mu1>
-      <mu2>2.0</mu2>
+        <mu1>1.0</mu1>
+        <mu2>1.0</mu2>
+        <kp>100000.0</kp>
+        <kd>10.0</kd>
+        <minDepth>0.001</minDepth>
+        <maxVel>0.1</maxVel>
+        <fdir1>1 0 0</fdir1>
     </gazebo>
     <gazebo reference="wheel_bl">
-      <mu1>2.0</mu1>
-      <mu2>2.0</mu2>
+        <mu1>1.0</mu1>
+        <mu2>1.0</mu2>
+        <kp>100000.0</kp>
+        <kd>10.0</kd>
+        <minDepth>0.001</minDepth>
+        <maxVel>0.1</maxVel>
+        <fdir1>1 0 0</fdir1>
     </gazebo>
     <gazebo reference="wheel_br">
-      <mu1>2.0</mu1>
-      <mu2>2.0</mu2>
+        <mu1>1.0</mu1>
+        <mu2>1.0</mu2>
+        <kp>100000.0</kp>
+        <kd>10.0</kd>
+        <minDepth>0.001</minDepth>
+        <maxVel>0.1</maxVel>
+        <fdir1>1 0 0</fdir1>
     </gazebo>
     <!-- ================= ACTUATOR LINKS ================= -->
@@ -34,7 +54,10 @@
     <!-- ================= ROS2 CONTROL (REQUIRED) ================= -->
     <gazebo>
-        <plugin filename="ign_ros2_control-system" name="ign_ros2_control::IgnitionROS2ControlPlugin">
-            <parameters>$(find sr_control)/config/runner_config.yaml</parameters>
-        </plugin>
+      <plugin filename="ign_ros2_control-system" name="ign_ros2_control::IgnitionROS2ControlPlugin">
+        <ros>
+          <namespace>$(arg namespace)</namespace>
+        </ros>
+        <parameters>$(find sr_control)/config/runner_config.yaml</parameters>
+      </plugin>
     </gazebo>
   </xacro:macro>

File: sr_description/urdf/wheel.urdf.xacro (robot description, xacro)
@@ -12,16 +12,8 @@
       <collision>
         <!-- Cylinder axis along X (wheel rotation axis) -->
-        <origin rpy="1.5708 0 0"/>
+        <origin xyz="0 0 0" rpy="0 0 0"/>
         <geometry>
-          <cylinder radius="0.05" length="0.04"/>
+            <sphere radius="0.05"/>
         </geometry>
-        <surface>
-          <friction>
-            <ode>
-              <mu>2.0</mu>
-              <mu2>2.0</mu2>
-            </ode>
-          </friction>
-        </surface>
       </collision>
       <inertial>
@@ -44,4 +36,5 @@
       <!-- Rotation around X axis -->
       <axis xyz="0 ${axis}  0"/>
+      <limit effort="100.0" velocity="40.0" />
     </joint>
   </xacro:macro>

Commit message: algorithm draft -1

File: sr_description/urdf/base.urdf.xacro (robot description, xacro)
@@ -41,4 +41,10 @@
         </geometry>
       </visual>
+      <collision>
+        <geometry>
+          <mesh filename="package://sr_description/meshes/wheel_shaft.stl"
+                scale="0.002 0.002 0.002"/>
+        </geometry>
+      </collision>
     </link>
     <joint name="shaft_fl_joint" type="fixed">
@@ -55,4 +61,10 @@
         </geometry>
       </visual>
+      <collision>
+        <geometry>
+          <mesh filename="package://sr_description/meshes/wheel_shaft.stl"
+                scale="0.002 0.002 0.002"/>
+        </geometry>
+      </collision>
     </link>
     <joint name="shaft_fr_joint" type="fixed">
@@ -69,4 +81,10 @@
         </geometry>
       </visual>
+      <collision>
+        <geometry>
+          <mesh filename="package://sr_description/meshes/wheel_shaft.stl"
+                scale="0.002 0.002 0.002"/>
+        </geometry>
+      </collision>
     </link>
     <joint name="shaft_bl_joint" type="fixed">
@@ -83,4 +101,10 @@
         </geometry>
       </visual>
+      <collision>
+        <geometry>
+          <mesh filename="package://sr_description/meshes/wheel_shaft.stl"
+                scale="0.002 0.002 0.002"/>
+        </geometry>
+      </collision>
     </link>
     <joint name="shaft_br_joint" type="fixed">

File: sr_description/urdf/wheel.urdf.xacro (robot description, xacro)
@@ -14,5 +14,5 @@
         <origin xyz="0 0 0" rpy="0 0 0"/>
         <geometry>
-            <sphere radius="0.05"/>
+          <mesh filename="package://sr_description/meshes/${mesh}" scale="0.0018 0.0018 0.0018"/>
         </geometry>
       </collision>
@@ -45,5 +45,5 @@
       mesh="mecanum_wheel_left.stl"
       shaft_link="shaft_fl"
-      offset="0.05"
+      offset="0.1"
       axis="1"/>
     <!-- Front Right -->
@@ -52,5 +52,5 @@
       mesh="mecanum_wheel_right.stl"
       shaft_link="shaft_fr"
-      offset="0.05"
+      offset="0.1"
       axis="-1"/>
     <!-- Back Left -->
@@ -59,5 +59,5 @@
       mesh="mecanum_wheel_right.stl"
       shaft_link="shaft_bl"
-      offset="0.05"
+      offset="0.1"
       axis="1"/>
     <!-- Back Right -->
@@ -66,5 +66,5 @@
       mesh="mecanum_wheel_left.stl"
       shaft_link="shaft_br"
-      offset="0.05"
+      offset="0.1"
       axis="-1"/>
   </xacro:macro>
