Commit message: urdf draft-4

File: sr_description/urdf/base.urdf.xacro (robot description, xacro)
@@ -9,5 +9,5 @@
         <origin xyz="0 0 0"/>
         <geometry>
-          <box size="0.44 0.36 0.1"/>
+          <box size="0.40 0.32 0.1"/>
         </geometry>
         <material name="grey"/>
@@ -16,5 +16,5 @@
         <origin xyz="0 0 0"/>
         <geometry>
-          <box size="0.44 0.36 0.1"/>
+          <box size="0.40 0.32 0.1"/>
         </geometry>
       </collision>
@@ -32,85 +32,4 @@
       <origin xyz="0 0 0.05"/>
     </joint>
-    <!-- ================= SHAFT LINKS ================= -->
-    <!-- Shaft FL -->
-    <link name="shaft_fl">
-      <visual>
-        <geometry>
-          <mesh filename="package://sr_description/meshes/wheel_shaft.stl"
-                scale="0.002 0.002 0.002"/>
-        </geometry>
-      </visual>
-      <collision>
-        <geometry>
-          <mesh filename="package://sr_description/meshes/wheel_shaft.stl"
-                scale="0.002 0.002 0.002"/>
-        </geometry>
-      </collision>
-    </link>
-    <joint name="shaft_fl_joint" type="fixed">
-      <parent link="base_link"/>
-      <child link="shaft_fl"/>
-      <origin xyz="0.20 0.18 0.0"/>
-    </joint>
-    <!-- Shaft FR -->
-    <link name="shaft_fr">
-      <visual>
-        <geometry>
-          <mesh filename="package://sr_description/meshes/wheel_shaft.stl"
-                scale="0.002 0.002 0.002"/>
-        </geometry>
-      </visual>
-      <collision>
-        <geometry>
-          <mesh filename="package://sr_description/meshes/wheel_shaft.stl"
-                scale="0.002 0.002 0.002"/>
-        </geometry>
-      </collision>
-    </link>
-    <joint name="shaft_fr_joint" type="fixed">
-      <parent link="base_link"/>
-      <child link="shaft_fr"/>
-      <origin xyz="0.20 -0.18 0.0" rpy="0 0 3.1416"/>
-    </joint>
-    <!-- Shaft BL -->
-    <link name="shaft_bl">
-      <visual>
-        <geometry>
-          <mesh filename="package://sr_description/meshes/wheel_shaft.stl"
-                scale="0.002 0.002 0.002"/>
-        </geometry>
-      </visual>
-      <collision>
-        <geometry>
-          <mesh filename="package://sr_description/meshes/wheel_shaft.stl"
-                scale="0.002 0.002 0.002"/>
-        </geometry>
-      </collision>
-    </link>
-    <joint name="shaft_bl_joint" type="fixed">
-      <parent link="base_link"/>
-      <child link="shaft_bl"/>
-      <origin xyz="-0.20 0.18 0.0"/>
-    </joint>
-    <!-- Shaft BR -->
-    <link name="shaft_br">
-      <visual>
-        <geometry>
-          <mesh filename="package://sr_description/meshes/wheel_shaft.stl"
-                scale="0.002 0.002 0.002"/>
-        </geometry>
-      </visual>
-      <collision>
-        <geometry>
-          <mesh filename="package://sr_description/meshes/wheel_shaft.stl"
-                scale="0.002 0.002 0.002"/>
-        </geometry>
-      </collision>
-    </link>
-    <joint name="shaft_br_joint" type="fixed">
-      <parent link="base_link"/>
-      <child link="shaft_br"/>
-      <origin xyz="-0.20 -0.18 0.0" rpy="0 0 3.1416"/>
-    </joint>
     <!-- ================= ARM MOUNT ================= -->
     <link name="arm_base_link"/>

File: sr_description/urdf/lifter_gazebo.urdf.xacro (robot description, xacro)
@@ -42,28 +42,29 @@
         <fdir1>1 1 0</fdir1>
     </gazebo>
+    <!-- Joint State Publisher -->
     <gazebo>
-      <plugin filename="ignition-gazebo-joint-controller-system" name="ignition::gazebo::systems::JointController">
-        <joint_name>wheel_fl_joint</joint_name>
-        <topic>/${robot_ns}/cmd_wheel_fl</topic>
+      <plugin filename="libignition-gazebo6-joint-state-publisher-system.so" name="ignition::gazebo::systems::JointStatePublisher">
       </plugin>
-      <plugin filename="ignition-gazebo-joint-controller-system" name="ignition::gazebo::systems::JointController">
-        <joint_name>wheel_fr_joint</joint_name>
-        <topic>/${robot_ns}/cmd_wheel_fr</topic>
-      </plugin>
-      <plugin filename="ignition-gazebo-joint-controller-system" name="ignition::gazebo::systems::JointController">
-        <joint_name>wheel_bl_joint</joint_name>
-        <topic>/${robot_ns}/cmd_wheel_bl</topic>
-      </plugin>
-      <plugin filename="ignition-gazebo-joint-controller-system" name="ignition::gazebo::systems::JointController">
-        <joint_name>wheel_br_joint</joint_name>
-        <topic>/${robot_ns}/cmd_wheel_br</topic>
+    </gazebo>
+    <!-- Mecanum Drive Plugin - Handles all wheels and kinematics! -->
+    <gazebo>
+      <plugin filename="libignition-gazebo6-mecanum-drive-system.so" name="ignition::gazebo::systems::MecanumDrive">
+        <front_left_joint>wheel_fl_joint</front_left_joint>
+        <front_right_joint>wheel_fr_joint</front_right_joint>
+        <back_left_joint>wheel_bl_joint</back_left_joint>
+        <back_right_joint>wheel_br_joint</back_right_joint>
+        <wheel_separation>0.4</wheel_separation>
+        <wheel_diameter>0.2</wheel_diameter>
+        <max_linear_speed>5.0</max_linear_speed>
+        <max_angular_speed>5.0</max_angular_speed>
+        <topic>${robot_ns}/cmd_vel</topic>
       </plugin>
     </gazebo>
     <gazebo>
-      <plugin filename="ignition-gazebo-joint-controller-system" name="ignition::gazebo::systems::JointController">
+      <plugin filename="libignition-gazebo6-joint-controller-system.so" name="ignition::gazebo::systems::JointController">
         <joint_name>arm_joint_1</joint_name>
         <topic>/${robot_ns}/cmd_shoulder</topic>
       </plugin>
-      <plugin filename="ignition-gazebo-joint-controller-system" name="ignition::gazebo::systems::JointController">
+      <plugin filename="libignition-gazebo6-joint-controller-system.so" name="ignition::gazebo::systems::JointController">
         <joint_name>arm_joint_2</joint_name>
         <topic>/${robot_ns}/cmd_elbow</topic>
@@ -71,9 +72,9 @@
     </gazebo>
     <gazebo>
-      <plugin filename="ignition-gazebo-odometry-publisher-system" name="ignition::gazebo::systems::OdometryPublisher">
-        <odom_frame>odom</odom_frame>
-        <robot_base_frame>${robot_ns}/base_footprint</robot_base_frame>
-        <odom_topic>/${robot_ns}/odom</odom_topic>
-        <tf_topic>/${robot_ns}/tf</tf_topic>
+      <plugin filename="libignition-gazebo6-odometry-publisher-system.so" name="ignition::gazebo::systems::OdometryPublisher">
+        <body_name>base_link</body_name>
+        <odom_publish_frequency>100</odom_publish_frequency>
+        <odom_topic>${robot_ns}/odom</odom_topic>
+        <tf_topic>${robot_ns}/tf</tf_topic>
       </plugin>
     </gazebo>

File: sr_description/urdf/runner_gazebo.urdf.xacro (robot description, xacro)
@@ -42,24 +42,25 @@
         <fdir1>1 1 0</fdir1>
     </gazebo>
+    <!-- Joint State Publisher -->
     <gazebo>
-      <plugin filename="ignition-gazebo-joint-controller-system" name="ignition::gazebo::systems::JointController">
-        <joint_name>wheel_fl_joint</joint_name>
-        <topic>/${robot_ns}/cmd_wheel_fl</topic>
+      <plugin filename="libignition-gazebo6-joint-state-publisher-system.so" name="ignition::gazebo::systems::JointStatePublisher">
       </plugin>
-      <plugin filename="ignition-gazebo-joint-controller-system" name="ignition::gazebo::systems::JointController">
-        <joint_name>wheel_fr_joint</joint_name>
-        <topic>/${robot_ns}/cmd_wheel_fr</topic>
-      </plugin>
-      <plugin filename="ignition-gazebo-joint-controller-system" name="ignition::gazebo::systems::JointController">
-        <joint_name>wheel_bl_joint</joint_name>
-        <topic>/${robot_ns}/cmd_wheel_bl</topic>
-      </plugin>
-      <plugin filename="ignition-gazebo-joint-controller-system" name="ignition::gazebo::systems::JointController">
-        <joint_name>wheel_br_joint</joint_name>
-        <topic>/${robot_ns}/cmd_wheel_br</topic>
+    </gazebo>
+    <!-- Mecanum Drive Plugin - Handles all wheels and kinematics! -->
+    <gazebo>
+      <plugin filename="libignition-gazebo6-mecanum-drive-system.so" name="ignition::gazebo::systems::MecanumDrive">
+        <front_left_joint>wheel_fl_joint</front_left_joint>
+        <front_right_joint>wheel_fr_joint</front_right_joint>
+        <back_left_joint>wheel_bl_joint</back_left_joint>
+        <back_right_joint>wheel_br_joint</back_right_joint>
+        <wheel_separation>0.4</wheel_separation>
+        <wheel_diameter>0.2</wheel_diameter>
+        <max_linear_speed>5.0</max_linear_speed>
+        <max_angular_speed>5.0</max_angular_speed>
+        <topic>${robot_ns}/cmd_vel</topic>
       </plugin>
     </gazebo>
     <gazebo>
-      <plugin filename="ignition-gazebo-joint-controller-system" name="ignition::gazebo::systems::JointController">
+      <plugin filename="libignition-gazebo6-joint-controller-system.so" name="ignition::gazebo::systems::JointController">
         <joint_name>piston_rod_joint</joint_name>
         <topic>/${robot_ns}/cmd_piston</topic>
@@ -67,9 +68,9 @@
     </gazebo>
     <gazebo>
-      <plugin filename="ignition-gazebo-odometry-publisher-system" name="ignition::gazebo::systems::OdometryPublisher">
-        <odom_frame>odom</odom_frame>
-        <robot_base_frame>${robot_ns}/base_footprint</robot_base_frame>
-        <odom_topic>/${robot_ns}/odom</odom_topic>
-        <tf_topic>/${robot_ns}/tf</tf_topic>
+      <plugin filename="libignition-gazebo6-odometry-publisher-system.so" name="ignition::gazebo::systems::OdometryPublisher">
+        <body_name>base_link</body_name>
+        <odom_publish_frequency>100</odom_publish_frequency>
+        <odom_topic>${robot_ns}/odom</odom_topic>
+        <tf_topic>${robot_ns}/tf</tf_topic>
       </plugin>
     </gazebo>

File: sr_description/urdf/wheel.urdf.xacro (robot description, xacro)
@@ -1,71 +1,125 @@
 <?xml version="1.0"?>
 <robot xmlns:xacro="http://www.ros.org/wiki/xacro">
-  <xacro:macro name="mecanum_wheel" params="name mesh shaft_link offset axis">
-    <link name="${name}">
+  <xacro:macro name="create_wheels">
+    <!-- ================= FRONT LEFT WHEEL ================= -->
+    <link name="wheel_fl_link">
       <visual>
-        <origin rpy="0 0 0"/>
+        <origin xyz="0 0 0" rpy="1.5708 0 0"/>
         <geometry>
-          <mesh filename="package://sr_description/meshes/${mesh}" scale="0.0018 0.0018 0.0018"/>
+          <cylinder radius="0.1" length="0.08"/>
         </geometry>
         <material name="dark_grey"/>
       </visual>
       <collision>
-        <!-- Cylinder axis along X (wheel rotation axis) -->
-        <origin xyz="0 0 0" rpy="0 0 0"/>
+        <origin xyz="0 0 0" rpy="1.5708 0 0"/>
         <geometry>
-          <mesh filename="package://sr_description/meshes/${mesh}" scale="0.0018 0.0018 0.0018"/>
+          <cylinder radius="0.1" length="0.08"/>
         </geometry>
       </collision>
       <inertial>
-        <origin rpy="0 0 0"/>
+        <origin xyz="0 0 0"/>
         <mass value="0.5"/>
-        <inertia
-          ixx="0.001"
-          iyy="0.001"
-          izz="0.001"
-          ixy="0"
-          ixz="0"
-          iyz="0"/>
+        <inertia ixx="0.001" iyy="0.001" izz="0.001" ixy="0" ixz="0" iyz="0"/>
       </inertial>
     </link>
-    <joint name="${name}_joint" type="continuous">
-      <parent link="${shaft_link}"/>
-      <child link="${name}"/>
-      <!-- Offset outward from shaft -->
-      <origin xyz="0 ${offset} 0"/>
-      <!-- Rotation around X axis -->
-      <axis xyz="0 ${axis}  0"/>
-      <limit effort="100.0" velocity="40.0" />
+    <!-- Front Left Joint - DIRECTLY TO BASE_LINK -->
+    <joint name="wheel_fl_joint" type="revolute">
+      <parent link="base_link"/>
+      <child link="wheel_fl_link"/>
+      <origin xyz="0.20 0.20 0.0" rpy="0 0 0"/>
+      <axis xyz="0 1 0"/>
+      <limit effort="100.0" velocity="40.0" lower="-3.14159" upper="3.14159"/>
+      <dynamics damping="0.1" friction="0.1"/>
+    </joint>
+    <!-- ================= FRONT RIGHT WHEEL ================= -->
+    <link name="wheel_fr_link">
+      <visual>
+        <origin xyz="0 0 0" rpy="1.5708 0 0"/>
+        <geometry>
+          <cylinder radius="0.1" length="0.08"/>
+        </geometry>
+        <material name="dark_grey"/>
+      </visual>
+      <collision>
+        <origin xyz="0 0 0" rpy="1.5708 0 0"/>
+        <geometry>
+          <cylinder radius="0.1" length="0.08"/>
+        </geometry>
+      </collision>
+      <inertial>
+        <origin xyz="0 0 0"/>
+        <mass value="0.5"/>
+        <inertia ixx="0.001" iyy="0.001" izz="0.001" ixy="0" ixz="0" iyz="0"/>
+      </inertial>
+    </link>
+    <!-- Front Right Joint - DIRECTLY TO BASE_LINK -->
+    <joint name="wheel_fr_joint" type="revolute">
+      <parent link="base_link"/>
+      <child link="wheel_fr_link"/>
+      <origin xyz="0.20 -0.20 0.0" rpy="0 0 0"/>
+      <axis xyz="0 1 0"/>
+      <limit effort="100.0" velocity="40.0" lower="-3.14159" upper="3.14159"/>
+      <dynamics damping="0.1" friction="0.1"/>
+    </joint>
+    <!-- ================= REAR LEFT WHEEL ================= -->
+    <link name="wheel_bl_link">
+      <visual>
+        <origin xyz="0 0 0" rpy="1.5708 0 0"/>
+        <geometry>
+          <cylinder radius="0.1" length="0.08"/>
+        </geometry>
+        <material name="dark_grey"/>
+      </visual>
+      <collision>
+        <origin xyz="0 0 0" rpy="1.5708 0 0"/>
+        <geometry>
+          <cylinder radius="0.1" length="0.08"/>
+        </geometry>
+      </collision>
+      <inertial>
+        <origin xyz="0 0 0"/>
+        <mass value="0.5"/>
+        <inertia ixx="0.001" iyy="0.001" izz="0.001" ixy="0" ixz="0" iyz="0"/>
+      </inertial>
+    </link>
+    <!-- Rear Left Joint - DIRECTLY TO BASE_LINK -->
+    <joint name="wheel_bl_joint" type="revolute">
+      <parent link="base_link"/>
+      <child link="wheel_bl_link"/>
+      <origin xyz="-0.20 0.20 0.0" rpy="0 0 0"/>
+      <axis xyz="0 1 0"/>
+      <limit effort="100.0" velocity="40.0" lower="-3.14159" upper="3.14159"/>
+      <dynamics damping="0.1" friction="0.1"/>
+    </joint>
+    <!-- ================= REAR RIGHT WHEEL ================= -->
+    <link name="wheel_br_link">
+      <visual>
+        <origin xyz="0 0 0" rpy="1.5708 0 0"/>
+        <geometry>
+          <cylinder radius="0.1" length="0.08"/>
+        </geometry>
+        <material name="dark_grey"/>
+      </visual>
+      <collision>
+        <origin xyz="0 0 0" rpy="1.5708 0 0"/>
+        <geometry>
+          <cylinder radius="0.1" length="0.08"/>
+        </geometry>
+      </collision>
+      <inertial>
+        <origin xyz="0 0 0"/>
+        <mass value="0.5"/>
+        <inertia ixx="0.001" iyy="0.001" izz="0.001" ixy="0" ixz="0" iyz="0"/>
+      </inertial>
+    </link>
+    <!-- Rear Right Joint - DIRECTLY TO BASE_LINK -->
+    <joint name="wheel_br_joint" type="revolute">
+      <parent link="base_link"/>
+      <child link="wheel_br_link"/>
+      <origin xyz="-0.20 -0.20 0.0" rpy="0 0 0"/>
+      <axis xyz="0 1 0"/>
+      <limit effort="100.0" velocity="40.0" lower="-3.14159" upper="3.14159"/>
+      <dynamics damping="0.1" friction="0.1"/>
     </joint>
   </xacro:macro>
-  <xacro:macro name="create_wheels">
-    <!-- Front Left -->
-    <xacro:mecanum_wheel
-      name="wheel_fl"
-      mesh="mecanum_wheel_left.stl"
-      shaft_link="shaft_fl"
-      offset="0.1"
-      axis="1"/>
-    <!-- Front Right -->
-    <xacro:mecanum_wheel
-      name="wheel_fr"
-      mesh="mecanum_wheel_right.stl"
-      shaft_link="shaft_fr"
-      offset="0.1"
-      axis="-1"/>
-    <!-- Back Left -->
-    <xacro:mecanum_wheel
-      name="wheel_bl"
-      mesh="mecanum_wheel_right.stl"
-      shaft_link="shaft_bl"
-      offset="0.1"
-      axis="1"/>
-    <!-- Back Right -->
-    <xacro:mecanum_wheel
-      name="wheel_br"
-      mesh="mecanum_wheel_left.stl"
-      shaft_link="shaft_br"
-      offset="0.1"
-      axis="-1"/>
-  </xacro:macro>
 </robot>
