Commit message: urdf draft-2

File: sr_description/urdf/actuator.urdf.xacro (robot description, xacro)
@@ -1,51 +1,47 @@
 <?xml version="1.0"?>
 <robot xmlns:xacro="http://www.ros.org/wiki/xacro" name="piston">
-  <!-- ========================================
-       PISTON ACTUATOR - MOUNTED ON WALL
-       Pushes box that sits on top of bot
-       ======================================== -->
   <!-- Piston parameters -->
-  <xacro:property name="piston_base_length" value="0.07"/>    <!-- Retracted length -->
-  <xacro:property name="piston_rod_length" value="0.20"/>      <!-- Max extension -->
-  <xacro:property name="piston_rod_radius" value="0.015"/>     <!-- Rod diameter -->
-  <xacro:property name="piston_base_radius" value="0.025"/>    <!-- Base diameter -->
+  <xacro:property name="piston_base_length" value="0.05"/>
+  <xacro:property name="piston_rod_length" value="0.1"/>
+  <xacro:property name="piston_rod_radius" value="0.015"/>
+  <xacro:property name="piston_base_radius" value="0.025"/>
   <xacro:property name="piston_mass" value="2.0"/>
+  <xacro:property name="chassis_length" value="0.32"/>
   <xacro:macro name="create_piston">
-    <!-- ===== PISTON BASE (Fixed to wall) ===== -->
+    <!-- ================= BASE ================= -->
     <link name="piston_base">
       <inertial>
-        <origin xyz="0 0 0" rpy="0 0 0"/>
-        <mass value="0.5"/>
-        <inertia ixx="0.001" iyy="0.001" izz="0.001" ixy="0" ixz="0" iyz="0"/>
+        <origin xyz="0 0 0"/>
+        <mass value="0.3"/>
+        <inertia ixx="0.001" iyy="0.001" izz="0.001"
+                 ixy="0" ixz="0" iyz="0"/>
       </inertial>
-      <!-- Visual: Cylinder base (piston housing) -->
       <visual>
         <origin xyz="0 0 0" rpy="1.5708 0 0"/>
         <geometry>
-          <cylinder radius="${piston_base_radius}" length="${piston_base_length}"/>
+          <cylinder radius="${piston_base_radius}"
+                    length="${piston_base_length}"/>
         </geometry>
         <material name="dark_grey"/>
       </visual>
-      <!-- Collision: Same cylinder -->
       <collision>
         <origin xyz="0 0 0" rpy="1.5708 0 0"/>
         <geometry>
-          <cylinder radius="${piston_base_radius}" length="${piston_base_length}"/>
+          <cylinder radius="${piston_base_radius}"
+                    length="${piston_base_length}"/>
         </geometry>
       </collision>
     </link>
-    <!-- Mount piston base to wall -->
+    <!-- Fixed to wall -->
     <joint name="piston_base_joint" type="fixed">
       <parent link="back_wall"/>
       <child link="piston_base"/>
-      <!-- Center of wall, extends forward -->
-      <origin xyz="0 -0.15 0.06" rpy="0 0 0"/>
+      <origin xyz="0.01 -0.15 0.06"/>
     </joint>
-    <!-- ===== PISTON ROD (Moving part - extends/retracts) ===== -->
+    <!-- ================= ROD ================= -->
     <link name="piston_rod">
       <inertial>
         <origin xyz="${piston_rod_length/2} 0 0" rpy="0 0 0"/>
         <mass value="${piston_mass}"/>
-        <!-- Inertia for cylinder -->
         <inertia
           ixx="${piston_mass * piston_rod_radius * piston_rod_radius / 4}"
@@ -54,5 +50,5 @@
           ixy="0" ixz="0" iyz="0"/>
       </inertial>
-      <!-- Visual: Extendable rod -->
+      <!-- Rod starts at joint, extends forward -->
       <visual>
         <origin xyz="${piston_rod_length/2} 0 0" rpy="0 1.5708 0"/>
@@ -62,5 +58,4 @@
         <material name="black"/>
       </visual>
-      <!-- Collision: Same rod -->
       <collision>
         <origin xyz="${piston_rod_length/2} 0 0" rpy="0 1.5708 0"/>
@@ -70,46 +65,39 @@
       </collision>
     </link>
-    <!-- Prismatic joint: Piston rod slides in X direction -->
+    <!-- ================= PRISMATIC JOINT ================= -->
     <joint name="piston_rod_joint" type="prismatic">
       <parent link="piston_base"/>
       <child link="piston_rod"/>
-      <!-- Connects at base of piston housing -->
-      <origin xyz="0 0 0" rpy="0 0 0"/>
-      <!-- Moves along X axis (forward/backward) -->
+      <origin xyz="0 0 0"/>
       <axis xyz="1 0 0"/>
-      <!-- Min: retracted (0), Max: fully extended (rod_length) -->
-      <limit lower="0" upper="${piston_rod_length}" effort="100" velocity="0.5"/>
-      <!-- Damping and friction for smooth motion -->
+      <!-- Starts retracted at 0 -->
+      <limit lower="0" upper="${chassis_length}"
+             effort="100" velocity="0.5"/>
       <dynamics damping="10" friction="0.5"/>
     </joint>
-    <!-- ===== PISTON HEAD (Pusher plate - at tip of rod) ===== -->
+    <!-- ================= PUSHER HEAD ================= -->
     <link name="piston_head">
       <inertial>
-        <origin xyz="0 0 0" rpy="0 0 0"/>
+        <origin xyz="0 0 0"/>
         <mass value="0.5"/>
-        <inertia ixx="0.001" iyy="0.001" izz="0.001" ixy="0" ixz="0" iyz="0"/>
+        <inertia ixx="0.001" iyy="0.001" izz="0.001"
+                 ixy="0" ixz="0" iyz="0"/>
       </inertial>
-      <!-- Visual: Square pusher plate -->
       <visual>
-        <origin xyz="0 0 0" rpy="0 0 0"/>
         <geometry>
-          <!-- Square plate at tip of piston -->
-          <box size="0.10 0.20 0.05"/>
+          <box size="0.04 0.18 0.05"/>
         </geometry>
         <material name="red"/>
       </visual>
-      <!-- Collision: Plate for pushing box -->
       <collision>
-        <origin xyz="0 0 0" rpy="0 0 0"/>
         <geometry>
-          <box size="0.10 0.20 0.05"/>
+          <box size="0.04 0.18 0.05"/>
         </geometry>
       </collision>
     </link>
-    <!-- Piston head fixed to rod tip -->
+    <!-- Head at rod tip -->
     <joint name="piston_head_joint" type="fixed">
       <parent link="piston_rod"/>
       <child link="piston_head"/>
-      <!-- At the end of the rod -->
       <origin xyz="${piston_rod_length} 0 0" rpy="0 0 0"/>
     </joint>

File: sr_description/urdf/arm.urdf.xacro (robot description, xacro)
@@ -2,29 +2,73 @@
 <robot xmlns:xacro="http://www.ros.org/wiki/xacro">
   <xacro:macro name="create_arm">
+    <!-- ARM LINK 1 -->
     <link name="arm_link_1">
+      <!-- Inertia -->
+      <inertial>
+        <origin xyz="0 0 0.1" rpy="0 0 0"/>
+        <mass value="1.5"/>
+        <inertia
+          ixx="0.01" ixy="0.0" ixz="0.0"
+          iyy="0.01" iyz="0.0"
+          izz="0.01"/>
+      </inertial>
+      <!-- Visual -->
       <visual>
+        <origin xyz="0 0 0" rpy="0 0 0"/>
         <geometry>
-          <mesh filename="package://sr_description/meshes/arm_link.dae" scale = "5 5 5"/>
+          <mesh filename="package://sr_description/meshes/arm_link.dae"
+                scale="5 5 5"/>
         </geometry>
       </visual>
+      <!-- Collision (simple box for stability) -->
+      <collision>
+        <origin xyz="0 0 0.1" rpy="0 0 0"/>
+        <geometry>
+          <box size="0.05 0.05 0.25"/>
+        </geometry>
+      </collision>
     </link>
+    <!-- ARM LINK 2 -->
     <link name="arm_link_2">
+      <!-- Inertia -->
+      <inertial>
+        <origin xyz="0 0 0.1" rpy="0 0 0"/>
+        <mass value="1.0"/>
+        <inertia
+          ixx="0.005" ixy="0.0" ixz="0.0"
+          iyy="0.005" iyz="0.0"
+          izz="0.005"/>
+      </inertial>
+      <!-- Visual -->
       <visual>
+        <origin xyz="0 0 0" rpy="0 0 0"/>
         <geometry>
-          <mesh filename="package://sr_description/meshes/arm_elbow.dae" scale = "5 5 5"/>
+          <mesh filename="package://sr_description/meshes/arm_elbow.dae"
+                scale="5 5 5"/>
         </geometry>
       </visual>
+      <!-- Collision -->
+      <collision>
+        <origin xyz="0 0 0.1" rpy="0 0 0"/>
+        <geometry>
+          <box size="0.04 0.04 0.20"/>
+        </geometry>
+      </collision>
     </link>
+    <!-- JOINT 1 -->
     <joint name="arm_joint_1" type="continuous">
       <parent link="arm_base_link"/>
       <child link="arm_link_1"/>
-      <origin xyz="0 0 0"/>
+      <origin xyz="0 0 0" rpy="0 0 0"/>
       <axis xyz="0 1 0"/>
+      <dynamics damping="0.1" friction="0.1"/>
     </joint>
+    <!-- JOINT 2 -->
     <joint name="arm_joint_2" type="continuous">
       <parent link="arm_link_1"/>
       <child link="arm_link_2"/>
-      <origin xyz="0 0 0.22"/>
+      <origin xyz="0 0 0.22" rpy="0 0 0"/>
       <axis xyz="0 1 0"/>
+      <dynamics damping="0.1" friction="0.1"/>
     </joint>
   </xacro:macro>

File: sr_description/urdf/lifter_bot.urdf.xacro (robot description, xacro)
@@ -5,6 +5,8 @@
   <xacro:include filename="$(find sr_description)/urdf/wheel.urdf.xacro"/>
   <xacro:include filename="$(find sr_description)/urdf/arm.urdf.xacro"/>
+  <xacro:include filename="$(find sr_description)/urdf/lifter_gazebo.urdf.xacro"/>
   <xacro:create_base/>
   <xacro:create_wheels/>
   <xacro:create_arm/>
+  <xacro:gazebo_setup_lift/>
 </robot>

File: sr_description/urdf/runner_bot.urdf.xacro (robot description, xacro)
@@ -6,7 +6,9 @@
   <xacro:include filename="$(find sr_description)/urdf/actuator.urdf.xacro"/>
   <xacro:include filename="$(find sr_description)/urdf/wall.urdf.xacro"/>
+  <xacro:include filename="$(find sr_description)/urdf/runner_gazebo.urdf.xacro"/>
   <xacro:create_base/>
   <xacro:create_wheels/>
   <xacro:create_wall/>
   <xacro:create_piston/>
+  <xacro:gazebo_setup_run/>
 </robot>

File: sr_description/urdf/wheel.urdf.xacro (robot description, xacro)
@@ -30,8 +30,8 @@
   </xacro:macro>
   <xacro:macro name="create_wheels">
-    <xacro:mecanum_wheel name="wheel_fl" x="0.2" y="0.2" mesh="mecanum_wheel_left.STL"/>
-    <xacro:mecanum_wheel name="wheel_fr" x="0.2" y="-0.2" mesh="mecanum_wheel_right.STL"/>
-    <xacro:mecanum_wheel name="wheel_bl" x="-0.2" y="0.2" mesh="mecanum_wheel_right.STL"/>
-    <xacro:mecanum_wheel name="wheel_br" x="-0.2" y="-0.2" mesh="mecanum_wheel_left.STL"/>
+    <xacro:mecanum_wheel name="wheel_fl" x="0.2" y="0.2" mesh="mecanum_wheel_left.stl"/>
+    <xacro:mecanum_wheel name="wheel_fr" x="0.2" y="-0.2" mesh="mecanum_wheel_right.stl"/>
+    <xacro:mecanum_wheel name="wheel_bl" x="-0.2" y="0.2" mesh="mecanum_wheel_right.stl"/>
+    <xacro:mecanum_wheel name="wheel_br" x="-0.2" y="-0.2" mesh="mecanum_wheel_left.stl"/>
   </xacro:macro>
 </robot>

Commit message: debugging-1

File: sr_description/urdf/actuator.urdf.xacro (robot description, xacro)
@@ -80,5 +80,5 @@
       <inertial>
         <origin xyz="0 0 0"/>
-        <mass value="0.5"/>
+        <mass value="0.2"/>
         <inertia ixx="0.001" iyy="0.001" izz="0.001"
                  ixy="0" ixz="0" iyz="0"/>

File: sr_description/urdf/arm.urdf.xacro (robot description, xacro)
@@ -7,5 +7,5 @@
       <inertial>
         <origin xyz="0 0 0.1" rpy="0 0 0"/>
-        <mass value="1.5"/>
+        <mass value="0.5"/>
         <inertia
           ixx="0.01" ixy="0.0" ixz="0.0"
@@ -22,10 +22,10 @@
       </visual>
       <!-- Collision (simple box for stability) -->
-      <collision>
+      <!-- <collision>
         <origin xyz="0 0 0.1" rpy="0 0 0"/>
         <geometry>
-          <box size="0.05 0.05 0.25" scale="5 5 3"/>
+          <box size="0.05 0.05 0.15" scale="5 5 3"/>
         </geometry>
-      </collision>
+      </collision> -->
     </link>
     <!-- ARM LINK 2 -->
@@ -34,5 +34,5 @@
       <inertial>
         <origin xyz="0 0 0.1" rpy="0 0 0"/>
-        <mass value="1.0"/>
+        <mass value="0.35"/>
         <inertia
           ixx="0.005" ixy="0.0" ixz="0.0"
@@ -49,25 +49,27 @@
       </visual>
       <!-- Collision -->
-      <collision>
+      <!-- <collision>
         <origin xyz="0 0 0.1" rpy="0 0 0"/>
         <geometry>
-          <box size="0.04 0.04 0.20" scale="5 5 2"/>
+          <box size="0.04 0.04 0.10" scale="5 5 2"/>
         </geometry>
-      </collision>
+      </collision> -->
     </link>
     <!-- JOINT 1 -->
-    <joint name="arm_joint_1" type="continuous">
+    <joint name="arm_joint_1" type="revolute">
       <parent link="arm_base_link"/>
       <child link="arm_link_1"/>
       <origin xyz="0 0 0" rpy="0 0 0"/>
       <axis xyz="0 1 0"/>
+      <limit effort="100.0" velocity="10.0" lower="0.0" upper="1.5708"/>
       <dynamics damping="0.1" friction="0.1"/>
     </joint>
     <!-- JOINT 2 -->
-    <joint name="arm_joint_2" type="continuous">
+    <joint name="arm_joint_2" type="revolute">
       <parent link="arm_link_1"/>
       <child link="arm_link_2"/>
       <origin xyz="0 0 0.155" rpy="0 0 0"/>
       <axis xyz="0 1 0"/>
+      <limit effort="100.0" velocity="10.0" lower="0.0" upper="1.5708"/>
       <dynamics damping="0.1" friction="0.1"/>
     </joint>

File: sr_description/urdf/lifter_gazebo.urdf.xacro (robot description, xacro)
@@ -3,27 +3,56 @@
   <xacro:macro name="gazebo_setup_lift" params="robot_ns">
     <gazebo>
-        <plugin
-        filename="ignition-gazebo-velocity-control-system"
-        name="gz::sim::systems::VelocityControl">
-        </plugin>
-        <plugin filename="ignition-gazebo-joint-state-publisher-system"
-        name="ignition::gazebo::systems::JointStatePublisher">
-        </plugin>
-        <!-- ign topic -t "/model/{bot_name}/joint/arm_base/cmd_vel" -m ignition.msgs.Double -p "data: 10.0" -->
-        <plugin filename="ignition-gazebo-joint-controller-system"
-        name="gz::sim::systems::JointController">
-        <joint_name>arm_joint_1</joint_name>
-        </plugin>
-        <plugin filename="ignition-gazebo-joint-controller-system"
-        name="gz::sim::systems::JointController">
-        <joint_name>arm_joint_2</joint_name>
-        </plugin>
-        <plugin filename="libignition-gazebo6-odometry-publisher-system.so"
-        name="ignition::gazebo::systems::OdometryPublisher">
-          <body_name>base_link</body_name>
-          <odom_publish_frequency>100</odom_publish_frequency>
-          <odom_topic>${robot_ns}/odom</odom_topic>
-          <tf_topic>${robot_ns}/tf</tf_topic>
-        </plugin>
+        <static>false</static>
+    </gazebo>
+    <gazebo reference="wheel_fl_link">
+      <mu1>5.0</mu1>      <!-- INCREASE friction -->
+      <mu2>5.0</mu2>      <!-- INCREASE friction -->
+      <kp>10000000.0</kp> <!-- INCREASE stiffness -->
+      <kd>1000.0</kd>     <!-- INCREASE damping -->
+    </gazebo>
+    <gazebo reference="wheel_fr_link">
+      <mu1>5.0</mu1>      <!-- INCREASE friction -->
+      <mu2>5.0</mu2>      <!-- INCREASE friction -->
+      <kp>10000000.0</kp> <!-- INCREASE stiffness -->
+      <kd>1000.0</kd>     <!-- INCREASE damping -->
+    </gazebo>
+    <gazebo reference="wheel_bl_link">
+      <mu1>5.0</mu1>      <!-- INCREASE friction -->
+      <mu2>5.0</mu2>      <!-- INCREASE friction -->
+      <kp>10000000.0</kp> <!-- INCREASE stiffness -->
+      <kd>1000.0</kd>     <!-- INCREASE damping -->
+    </gazebo>
+    <gazebo reference="wheel_br_link">
+      <mu1>5.0</mu1>      <!-- INCREASE friction -->
+      <mu2>5.0</mu2>      <!-- INCREASE friction -->
+      <kp>10000000.0</kp> <!-- INCREASE stiffness -->
+      <kd>1000.0</kd>     <!-- INCREASE damping -->
+    </gazebo>
+    <gazebo>
+      <plugin filename="libignition-gazebo-joint-state-publisher-system.so"
+              name="ignition::gazebo::systems::JointStatePublisher">
+      </plugin>
+      <plugin filename="libignition-gazebo-joint-controller-system.so" name="ignition::gazebo::systems::JointController">
+          <joint_name>wheel_fl_joint</joint_name>
+          <cmd_vel_topic>/model/lifter1/joint/wheel_fl_joint/cmd_vel</cmd_vel_topic>
+      </plugin>
+      <plugin filename="libignition-gazebo-joint-controller-system.so" name="ignition::gazebo::systems::JointController">
+          <joint_name>wheel_fr_joint</joint_name>
+          <cmd_vel_topic>/model/lifter1/joint/wheel_fr_joint/cmd_vel</cmd_vel_topic>
+      </plugin>
+      <plugin filename="libignition-gazebo-joint-controller-system.so" name="ignition::gazebo::systems::JointController">
+          <joint_name>wheel_bl_joint</joint_name>
+          <cmd_vel_topic>/model/lifter1/joint/wheel_bl_joint/cmd_vel</cmd_vel_topic>
+      </plugin>
+      <plugin filename="libignition-gazebo-joint-controller-system.so" name="ignition::gazebo::systems::JointController">
+          <joint_name>wheel_br_joint</joint_name>
+          <cmd_vel_topic>/model/lifter1/joint/wheel_br_joint/cmd_vel</cmd_vel_topic>
+      </plugin>
+      <plugin filename="libignition-gazebo-odometry-publisher-system.so" name="ignition::gazebo::systems::OdometryPublisher">
+          <odom_cmd_vel_topic>/lifter1/odom</odom_cmd_vel_topic>
+          <odom_frame>odom</odom_frame>
+          <robot_base_frame>base_footprint</robot_base_frame>
+          <odom_publish_frequency>50</odom_publish_frequency>
+      </plugin>
     </gazebo>
   </xacro:macro>

File: sr_description/urdf/runner_gazebo.urdf.xacro (robot description, xacro)
@@ -3,23 +3,56 @@
   <xacro:macro name="gazebo_setup_run" params="robot_ns">
     <gazebo>
-        <plugin
-        filename="ignition-gazebo-velocity-control-system"
-        name="gz::sim::systems::VelocityControl">
-        </plugin>
-        <plugin filename="ignition-gazebo-joint-state-publisher-system"
-        name="ignition::gazebo::systems::JointStatePublisher">
-        </plugin>
-        <!-- ign topic -t "/model/{bot_name}/joint/arm_base/cmd_vel" -m ignition.msgs.Double -p "data: 10.0" -->
-        <plugin filename="ignition-gazebo-joint-controller-system"
-        name="gz::sim::systems::JointController">
-        <joint_name>piston_rod_joint</joint_name>
-        </plugin>
-        <plugin filename="libignition-gazebo6-odometry-publisher-system.so"
-        name="ignition::gazebo::systems::OdometryPublisher">
-          <body_name>base_link</body_name>
-          <odom_publish_frequency>100</odom_publish_frequency>
-          <odom_topic>${robot_ns}/odom</odom_topic>
-          <tf_topic>${robot_ns}/tf</tf_topic>
-        </plugin>
+        <static>false</static>
+    </gazebo>
+    <gazebo reference="wheel_fl_link">
+      <mu1>5.0</mu1>      <!-- INCREASE friction -->
+      <mu2>5.0</mu2>      <!-- INCREASE friction -->
+      <kp>10000000.0</kp> <!-- INCREASE stiffness -->
+      <kd>1000.0</kd>     <!-- INCREASE damping -->
+    </gazebo>
+    <gazebo reference="wheel_fr_link">
+      <mu1>5.0</mu1>      <!-- INCREASE friction -->
+      <mu2>5.0</mu2>      <!-- INCREASE friction -->
+      <kp>10000000.0</kp> <!-- INCREASE stiffness -->
+      <kd>1000.0</kd>     <!-- INCREASE damping -->
+    </gazebo>
+    <gazebo reference="wheel_bl_link">
+      <mu1>5.0</mu1>      <!-- INCREASE friction -->
+      <mu2>5.0</mu2>      <!-- INCREASE friction -->
+      <kp>10000000.0</kp> <!-- INCREASE stiffness -->
+      <kd>1000.0</kd>     <!-- INCREASE damping -->
+    </gazebo>
+    <gazebo reference="wheel_br_link">
+      <mu1>5.0</mu1>      <!-- INCREASE friction -->
+      <mu2>5.0</mu2>      <!-- INCREASE friction -->
+      <kp>10000000.0</kp> <!-- INCREASE stiffness -->
+      <kd>1000.0</kd>     <!-- INCREASE damping -->
+    </gazebo>
+    <gazebo>
+      <plugin filename="libignition-gazebo-joint-state-publisher-system.so"
+              name="ignition::gazebo::systems::JointStatePublisher">
+      </plugin>
+      <plugin filename="libignition-gazebo-joint-controller-system.so" name="ignition::gazebo::systems::JointController">
+          <joint_name>wheel_fl_joint</joint_name>
+          <topic>/model/runner1/joint/wheel_fl_joint/cmd_vel</topic>
+      </plugin>
+      <plugin filename="libignition-gazebo-joint-controller-system.so" name="ignition::gazebo::systems::JointController">
+          <joint_name>wheel_fr_joint</joint_name>
+          <topic>/model/runner1/joint/wheel_fr_joint/cmd_vel</topic>
+      </plugin>
+      <plugin filename="libignition-gazebo-joint-controller-system.so" name="ignition::gazebo::systems::JointController">
+          <joint_name>wheel_bl_joint</joint_name>
+          <topic>/model/runner1/joint/wheel_bl_joint/cmd_vel</topic>
+      </plugin>
+      <plugin filename="libignition-gazebo-joint-controller-system.so" name="ignition::gazebo::systems::JointController">
+          <joint_name>wheel_br_joint</joint_name>
+          <topic>/model/runner1/joint/wheel_br_joint/cmd_vel</topic>
+      </plugin>
+      <plugin filename="libignition-gazebo-odometry-publisher-system.so" name="ignition::gazebo::systems::OdometryPublisher">
+          <odom_topic>/runner1/odom</odom_topic>
+          <odom_frame>odom</odom_frame>
+          <robot_base_frame>base_footprint</robot_base_frame>
+          <odom_publish_frequency>50</odom_publish_frequency>
+      </plugin>
     </gazebo>
   </xacro:macro>

File: sr_description/urdf/wheel.urdf.xacro (robot description, xacro)
@@ -3,4 +3,5 @@
   <xacro:macro name="create_wheels">
     <!-- ================= FRONT LEFT WHEEL ================= -->
+    <!-- Position: +X (front), +Y (left) -->
     <link name="wheel_fl_link">
       <visual>
@@ -23,5 +24,5 @@
       </inertial>
     </link>
-    <!-- Front Left Joint - DIRECTLY TO BASE_LINK -->
+    <!-- Front Left Joint -->
     <joint name="wheel_fl_joint" type="revolute">
       <parent link="base_link"/>
@@ -33,4 +34,5 @@
     </joint>
     <!-- ================= FRONT RIGHT WHEEL ================= -->
+    <!-- Position: +X (front), -Y (right) -->
     <link name="wheel_fr_link">
       <visual>
@@ -53,5 +55,5 @@
       </inertial>
     </link>
-    <!-- Front Right Joint - DIRECTLY TO BASE_LINK -->
+    <!-- Front Right Joint -->
     <joint name="wheel_fr_joint" type="revolute">
       <parent link="base_link"/>
@@ -63,4 +65,5 @@
     </joint>
     <!-- ================= REAR LEFT WHEEL ================= -->
+    <!-- Position: -X (back), +Y (left) -->
     <link name="wheel_bl_link">
       <visual>
@@ -83,5 +86,5 @@
       </inertial>
     </link>
-    <!-- Rear Left Joint - DIRECTLY TO BASE_LINK -->
+    <!-- Rear Left Joint -->
     <joint name="wheel_bl_joint" type="revolute">
       <parent link="base_link"/>
@@ -93,4 +96,5 @@
     </joint>
     <!-- ================= REAR RIGHT WHEEL ================= -->
+    <!-- Position: -X (back), -Y (right) -->
     <link name="wheel_br_link">
       <visual>
@@ -113,5 +117,5 @@
       </inertial>
     </link>
-    <!-- Rear Right Joint - DIRECTLY TO BASE_LINK -->
+    <!-- Rear Right Joint -->
     <joint name="wheel_br_joint" type="revolute">
       <parent link="base_link"/>
