Commit message: Gazebo spawn

File: sr_description/urdf/lifter_bot.urdf.xacro (robot description, xacro)
@@ -9,4 +9,4 @@
   <xacro:create_wheels/>
   <xacro:create_arm/>
-  <xacro:gazebo_setup_lift />
+  <xacro:gazebo_setup_lift robot_ns="lifter1" />
 </robot>

File: sr_description/urdf/lifter_gazebo.urdf.xacro (robot description, xacro)
@@ -1,11 +1,9 @@
 <?xml version="1.0"?>
 <robot xmlns:xacro="http://www.ros.org/wiki/xacro">
-  <xacro:macro name="gazebo_setup_lift">
-    <!-- ================= BASE ================= -->
+  <xacro:macro name="gazebo_setup_lift" params="robot_ns">
     <gazebo reference="base_link">
-      <mu1>0</mu1>
-      <mu2>0</mu2>
+      <mu1>0.2</mu1>
+      <mu2>0.2</mu2>
     </gazebo>
-    <!-- ================= MECANUM WHEELS ================= -->
     <gazebo reference="wheel_fl">
         <mu1>10.0</mu1>
@@ -44,18 +42,47 @@
         <fdir1>1 1 0</fdir1>
     </gazebo>
-    <!-- ================= ARM LINKS ================= -->
+    <gazebo>
+      <plugin filename="ignition-gazebo-joint-controller-system" name="ignition::gazebo::systems::JointController">
+        <joint_name>wheel_fl_joint</joint_name>
+        <topic>/${robot_ns}/cmd_wheel_fl</topic>
+      </plugin>
+      <plugin filename="ignition-gazebo-joint-controller-system" name="ignition::gazebo::systems::JointController">
+        <joint_name>wheel_fr_joint</joint_name>
+        <topic>/${robot_ns}/cmd_wheel_fr</topic>
+      </plugin>
+      <plugin filename="ignition-gazebo-joint-controller-system" name="ignition::gazebo::systems::JointController">
+        <joint_name>wheel_bl_joint</joint_name>
+        <topic>/${robot_ns}/cmd_wheel_bl</topic>
+      </plugin>
+      <plugin filename="ignition-gazebo-joint-controller-system" name="ignition::gazebo::systems::JointController">
+        <joint_name>wheel_br_joint</joint_name>
+        <topic>/${robot_ns}/cmd_wheel_br</topic>
+      </plugin>
+    </gazebo>
+    <gazebo>
+      <plugin filename="ignition-gazebo-joint-controller-system" name="ignition::gazebo::systems::JointController">
+        <joint_name>arm_joint_1</joint_name>
+        <topic>/${robot_ns}/cmd_shoulder</topic>
+      </plugin>
+      <plugin filename="ignition-gazebo-joint-controller-system" name="ignition::gazebo::systems::JointController">
+        <joint_name>arm_joint_2</joint_name>
+        <topic>/${robot_ns}/cmd_elbow</topic>
+      </plugin>
+    </gazebo>
+    <gazebo>
+      <plugin filename="ignition-gazebo-odometry-publisher-system" name="ignition::gazebo::systems::OdometryPublisher">
+        <odom_frame>odom</odom_frame>
+        <robot_base_frame>${robot_ns}/base_footprint</robot_base_frame>
+        <odom_topic>/${robot_ns}/odom</odom_topic>
+        <tf_topic>/${robot_ns}/tf</tf_topic>
+      </plugin>
+    </gazebo>
     <gazebo reference="arm_base_link"/>
-    <gazebo reference="arm_shoulder_link"/>
-    <gazebo reference="arm_elbow_link"/>
-    <gazebo reference="arm_wrist_link"/>
-    <gazebo reference="gripper_link"/>
-    <!-- ================= ARM JOINT DYNAMICS ================= -->
-    <gazebo reference="shoulder_joint">
+    <gazebo reference="arm_joint_1"/>
+    <gazebo reference="arm_joint_2"/>
+    <gazebo reference="arm_joint_1">
       <implicitSpringDamper>true</implicitSpringDamper>
     </gazebo>
-    <gazebo reference="elbow_joint">
-      <implicitSpringDamper>true</implicitSpringDamper>
-    </gazebo>
-    <gazebo reference="wrist_joint">
+    <gazebo reference="arm_joint_2">
       <implicitSpringDamper>true</implicitSpringDamper>
     </gazebo>

File: sr_description/urdf/runner_bot.urdf.xacro (robot description, xacro)
@@ -11,4 +11,4 @@
   <xacro:create_wall/>
   <xacro:create_piston/>
-  <xacro:gazebo_setup_run />
+  <xacro:gazebo_setup_run robot_ns="runner1"/>
 </robot>

File: sr_description/urdf/runner_gazebo.urdf.xacro (robot description, xacro)
@@ -1,46 +1,76 @@
 <?xml version="1.0"?>
 <robot xmlns:xacro="http://www.ros.org/wiki/xacro">
-  <xacro:macro name="gazebo_setup_run">
-    <!-- ================= BASE ================= -->
+  <xacro:macro name="gazebo_setup_run" params="robot_ns">
     <gazebo reference="base_link">
-      <mu1>0.3</mu1>
-      <mu2>0.3</mu2>
+      <mu1>0.2</mu1>
+      <mu2>0.2</mu2>
     </gazebo>
-    <!-- ================= MECANUM WHEELS ================= -->
     <gazebo reference="wheel_fl">
-        <mu1>1.0</mu1>
-        <mu2>1.0</mu2>
+        <mu1>10.0</mu1>
+        <mu2>10.0</mu2>
         <kp>100000.0</kp>
         <kd>10.0</kd>
         <minDepth>0.001</minDepth>
         <maxVel>0.1</maxVel>
-        <fdir1>1 0 0</fdir1>
+        <fdir1>1 1 0</fdir1>
     </gazebo>
     <gazebo reference="wheel_fr">
-        <mu1>1.0</mu1>
-        <mu2>1.0</mu2>
+        <mu1>10.0</mu1>
+        <mu2>10.0</mu2>
         <kp>100000.0</kp>
         <kd>10.0</kd>
         <minDepth>0.001</minDepth>
         <maxVel>0.1</maxVel>
-        <fdir1>1 0 0</fdir1>
+        <fdir1>1 -1 0</fdir1>
     </gazebo>
     <gazebo reference="wheel_bl">
-        <mu1>1.0</mu1>
-        <mu2>1.0</mu2>
+        <mu1>10.0</mu1>
+        <mu2>10.0</mu2>
         <kp>100000.0</kp>
         <kd>10.0</kd>
         <minDepth>0.001</minDepth>
         <maxVel>0.1</maxVel>
-        <fdir1>1 0 0</fdir1>
+        <fdir1>1 -1 0</fdir1>
     </gazebo>
     <gazebo reference="wheel_br">
-        <mu1>1.0</mu1>
-        <mu2>1.0</mu2>
+        <mu1>10.0</mu1>
+        <mu2>10.0</mu2>
         <kp>100000.0</kp>
         <kd>10.0</kd>
         <minDepth>0.001</minDepth>
         <maxVel>0.1</maxVel>
-        <fdir1>1 0 0</fdir1>
+        <fdir1>1 1 0</fdir1>
+    </gazebo>
+    <gazebo>
+      <plugin filename="ignition-gazebo-joint-controller-system" name="ignition::gazebo::systems::JointController">
+        <joint_name>wheel_fl_joint</joint_name>
+        <topic>/${robot_ns}/cmd_wheel_fl</topic>
+      </plugin>
+      <plugin filename="ignition-gazebo-joint-controller-system" name="ignition::gazebo::systems::JointController">
+        <joint_name>wheel_fr_joint</joint_name>
+        <topic>/${robot_ns}/cmd_wheel_fr</topic>
+      </plugin>
+      <plugin filename="ignition-gazebo-joint-controller-system" name="ignition::gazebo::systems::JointController">
+        <joint_name>wheel_bl_joint</joint_name>
+        <topic>/${robot_ns}/cmd_wheel_bl</topic>
+      </plugin>
+      <plugin filename="ignition-gazebo-joint-controller-system" name="ignition::gazebo::systems::JointController">
+        <joint_name>wheel_br_joint</joint_name>
+        <topic>/${robot_ns}/cmd_wheel_br</topic>
+      </plugin>
+    </gazebo>
+    <gazebo>
+      <plugin filename="ignition-gazebo-joint-controller-system" name="ignition::gazebo::systems::JointController">
+        <joint_name>piston_rod_joint</joint_name>
+        <topic>/${robot_ns}/cmd_piston</topic>
+      </plugin>
+    </gazebo>
+    <gazebo>
+      <plugin filename="ignition-gazebo-odometry-publisher-system" name="ignition::gazebo::systems::OdometryPublisher">
+        <odom_frame>odom</odom_frame>
+        <robot_base_frame>${robot_ns}/base_footprint</robot_base_frame>
+        <odom_topic>/${robot_ns}/odom</odom_topic>
+        <tf_topic>/${robot_ns}/tf</tf_topic>
+      </plugin>
     </gazebo>
     <!-- ================= ACTUATOR LINKS ================= -->
@@ -52,5 +82,4 @@
       <implicitSpringDamper>true</implicitSpringDamper>
     </gazebo>
-    <!-- ================= ROS2 CONTROL (REQUIRED) ================= -->
   </xacro:macro>
 </robot>

Commit message: complete draft-2

File: sr_description/urdf/lifter_bot.urdf.xacro (robot description, xacro)
@@ -1,4 +1,5 @@
 <?xml version="1.0"?>
 <robot xmlns:xacro="http://www.ros.org/wiki/xacro" name="lifter_bot">
+  <xacro:arg name="robot_ns" default="lifter1"/>
   <xacro:include filename="$(find sr_description)/urdf/material.urdf.xacro"/>
   <xacro:include filename="$(find sr_description)/urdf/base.urdf.xacro"/>
@@ -9,4 +10,4 @@
   <xacro:create_wheels/>
   <xacro:create_arm/>
-  <xacro:gazebo_setup_lift robot_ns="lifter1" />
+  <xacro:gazebo_setup_lift robot_ns="$(arg robot_ns)" />
 </robot>

File: sr_description/urdf/lifter_gazebo.urdf.xacro (robot description, xacro)
@@ -35,34 +35,32 @@
       <plugin filename="libignition-gazebo-joint-controller-system.so" name="ignition::gazebo::systems::JointController">
           <joint_name>wheel_fl_joint</joint_name>
-          <cmd_vel_topic>/model/lifter1/joint/wheel_fl_joint/cmd_vel</cmd_vel_topic>
+          <cmd_vel_topic>/model/${robot_ns}/joint/wheel_fl_joint/cmd_vel</cmd_vel_topic>
       </plugin>
       <plugin filename="libignition-gazebo-joint-controller-system.so" name="ignition::gazebo::systems::JointController">
           <joint_name>wheel_fr_joint</joint_name>
-          <cmd_vel_topic>/model/lifter1/joint/wheel_fr_joint/cmd_vel</cmd_vel_topic>
+          <cmd_vel_topic>/model/${robot_ns}/joint/wheel_fr_joint/cmd_vel</cmd_vel_topic>
       </plugin>
       <plugin filename="libignition-gazebo-joint-controller-system.so" name="ignition::gazebo::systems::JointController">
           <joint_name>wheel_bl_joint</joint_name>
-          <cmd_vel_topic>/model/lifter1/joint/wheel_bl_joint/cmd_vel</cmd_vel_topic>
+          <cmd_vel_topic>/model/${robot_ns}/joint/wheel_bl_joint/cmd_vel</cmd_vel_topic>
       </plugin>
       <plugin filename="libignition-gazebo-joint-controller-system.so" name="ignition::gazebo::systems::JointController">
           <joint_name>wheel_br_joint</joint_name>
-          <cmd_vel_topic>/model/lifter1/joint/wheel_br_joint/cmd_vel</cmd_vel_topic>
+          <cmd_vel_topic>/model/${robot_ns}/joint/wheel_br_joint/cmd_vel</cmd_vel_topic>
       </plugin>
       <plugin filename="libignition-gazebo-joint-controller-system.so"
               name="ignition::gazebo::systems::JointController">
           <joint_name>arm_joint_1</joint_name>
-          <cmd_vel_topic>/model/lifter1/joint/arm_joint_1/cmd_vel</cmd_vel_topic>
+          <cmd_vel_topic>/model/${robot_ns}/joint/arm_joint_1/cmd_vel</cmd_vel_topic>
       </plugin>
       <plugin filename="libignition-gazebo-joint-controller-system.so"
               name="ignition::gazebo::systems::JointController">
           <joint_name>arm_joint_2</joint_name>
-          <cmd_vel_topic>/model/lifter1/joint/arm_joint_2/cmd_vel</cmd_vel_topic>
+          <cmd_vel_topic>/model/${robot_ns}/joint/arm_joint_2/cmd_vel</cmd_vel_topic>
       </plugin>
-      <plugin
-        filename="libignition_link_attacher.so"
-        name="ignition_link_attacher">
+      <plugin filename="libignition_link_attacher.so" name="ignition_link_attacher">
       </plugin>
       <plugin filename="libignition-gazebo-odometry-publisher-system.so" name="ignition::gazebo::systems::OdometryPublisher">
-          <odom_topic>/lifter1/odom</odom_topic>
+          <odom_topic>/${robot_ns}/odom</odom_topic>
           <odom_frame>odom</odom_frame>
           <robot_base_frame>base_footprint</robot_base_frame>

File: sr_description/urdf/runner_bot.urdf.xacro (robot description, xacro)
@@ -1,14 +1,15 @@
 <?xml version="1.0"?>
 <robot xmlns:xacro="http://www.ros.org/wiki/xacro" name="runner_bot">
+  <xacro:arg name="robot_ns" default="runner1"/>
   <xacro:include filename="$(find sr_description)/urdf/material.urdf.xacro"/>
   <xacro:include filename="$(find sr_description)/urdf/base.urdf.xacro"/>
   <xacro:include filename="$(find sr_description)/urdf/wheel.urdf.xacro"/>
+  <xacro:include filename="$(find sr_description)/urdf/wall.urdf.xacro"/>
   <xacro:include filename="$(find sr_description)/urdf/actuator.urdf.xacro"/>
-  <xacro:include filename="$(find sr_description)/urdf/wall.urdf.xacro"/>
   <xacro:include filename="$(find sr_description)/urdf/runner_gazebo.urdf.xacro"/>
   <xacro:create_base/>
   <xacro:create_wheels/>
+  <xacro:create_piston/>
   <xacro:create_wall/>
-  <xacro:create_piston/>
-  <xacro:gazebo_setup_run robot_ns="runner1"/>
+  <xacro:gazebo_setup_runner robot_ns="$(arg robot_ns)" />
 </robot>

File: sr_description/urdf/runner_gazebo.urdf.xacro (robot description, xacro)
@@ -1,5 +1,5 @@
 <?xml version="1.0"?>
 <robot xmlns:xacro="http://www.ros.org/wiki/xacro">
-  <xacro:macro name="gazebo_setup_run" params="robot_ns">
+  <xacro:macro name="gazebo_setup_runner" params="robot_ns">
     <gazebo>
         <static>false</static>
@@ -35,29 +35,27 @@
       <plugin filename="libignition-gazebo-joint-controller-system.so" name="ignition::gazebo::systems::JointController">
           <joint_name>wheel_fl_joint</joint_name>
-          <topic>/model/runner1/joint/wheel_fl_joint/cmd_vel</topic>
+          <cmd_vel_topic>/model/${robot_ns}/joint/wheel_fl_joint/cmd_vel</cmd_vel_topic>
       </plugin>
       <plugin filename="libignition-gazebo-joint-controller-system.so" name="ignition::gazebo::systems::JointController">
           <joint_name>wheel_fr_joint</joint_name>
-          <topic>/model/runner1/joint/wheel_fr_joint/cmd_vel</topic>
+          <cmd_vel_topic>/model/${robot_ns}/joint/wheel_fr_joint/cmd_vel</cmd_vel_topic>
       </plugin>
       <plugin filename="libignition-gazebo-joint-controller-system.so" name="ignition::gazebo::systems::JointController">
           <joint_name>wheel_bl_joint</joint_name>
-          <topic>/model/runner1/joint/wheel_bl_joint/cmd_vel</topic>
+          <cmd_vel_topic>/model/${robot_ns}/joint/wheel_bl_joint/cmd_vel</cmd_vel_topic>
       </plugin>
       <plugin filename="libignition-gazebo-joint-controller-system.so" name="ignition::gazebo::systems::JointController">
           <joint_name>wheel_br_joint</joint_name>
-          <topic>/model/runner1/joint/wheel_br_joint/cmd_vel</topic>
-      </plugin>
-      <plugin
-        filename="libignition_link_attacher.so"
-        name="ignition_link_attacher">
+          <cmd_vel_topic>/model/${robot_ns}/joint/wheel_br_joint/cmd_vel</cmd_vel_topic>
       </plugin>
       <plugin filename="libignition-gazebo-joint-controller-system.so"
               name="ignition::gazebo::systems::JointController">
           <joint_name>piston_rod_joint</joint_name>
-          <cmd_vel_topic>/model/runner1/joint/piston_rod_joint/cmd_vel</cmd_vel_topic>
+          <cmd_vel_topic>/model/${robot_ns}/joint/piston_rod_joint/cmd_vel</cmd_vel_topic>
+      </plugin>
+      <plugin filename="libignition_link_attacher.so" name="ignition_link_attacher">
       </plugin>
       <plugin filename="libignition-gazebo-odometry-publisher-system.so" name="ignition::gazebo::systems::OdometryPublisher">
-          <odom_topic>/runner1/odom</odom_topic>
+          <odom_topic>/${robot_ns}/odom</odom_topic>
           <odom_frame>odom</odom_frame>
           <robot_base_frame>base_footprint</robot_base_frame>
