Commit message: setting up

File: sr_description/urdf/arm.urdf.xacro (robot description, xacro)
@@ -18,5 +18,5 @@
         <geometry>
           <mesh filename="package://sr_description/meshes/arm_link.dae"
-                scale="5 5 5"/>
+                scale="5 5 3"/>
         </geometry>
       </visual>
@@ -45,5 +45,5 @@
         <geometry>
           <mesh filename="package://sr_description/meshes/arm_elbow.dae"
-                scale="5 5 5"/>
+                scale="5 5 2"/>
         </geometry>
       </visual>
@@ -68,5 +68,5 @@
       <parent link="arm_link_1"/>
       <child link="arm_link_2"/>
-      <origin xyz="0 0 0.22" rpy="0 0 0"/>
+      <origin xyz="0 0 0.155" rpy="0 0 0"/>
       <axis xyz="0 1 0"/>
       <dynamics damping="0.1" friction="0.1"/>

File: sr_description/urdf/lifter_control.urdf.xacro (robot description, xacro)
@@ -45,4 +45,5 @@
     <joint name="arm_joint_1">
       <command_interface name="position"/>
+      <command_interface name="velocity"/>
       <state_interface name="position"/>
       <state_interface name="velocity"/>
@@ -50,4 +51,5 @@
     <joint name="arm_joint_2">
       <command_interface name="position"/>
+      <command_interface name="velocity"/>
       <state_interface name="position"/>
       <state_interface name="velocity"/>

File: sr_description/urdf/runner_control.urdf.xacro (robot description, xacro)
@@ -45,4 +45,5 @@
     <joint name="piston_rod_joint">
       <command_interface name="position"/>
+      <command_interface name="velocity"/>
       <state_interface name="position"/>
       <state_interface name="velocity"/>

Commit message: control draft-3

File: sr_description/urdf/arm.urdf.xacro (robot description, xacro)
@@ -25,5 +25,5 @@
         <origin xyz="0 0 0.1" rpy="0 0 0"/>
         <geometry>
-          <box size="0.05 0.05 0.25"/>
+          <box size="0.05 0.05 0.25" scale="5 5 3"/>
         </geometry>
       </collision>
@@ -52,5 +52,5 @@
         <origin xyz="0 0 0.1" rpy="0 0 0"/>
         <geometry>
-          <box size="0.04 0.04 0.20"/>
+          <box size="0.04 0.04 0.20" scale="5 5 2"/>
         </geometry>
       </collision>

File: sr_description/urdf/lifter_gazebo.urdf.xacro (robot description, xacro)
@@ -2,97 +2,28 @@
 <robot xmlns:xacro="http://www.ros.org/wiki/xacro">
   <xacro:macro name="gazebo_setup_lift" params="robot_ns">
-    <gazebo reference="base_link">
-      <mu1>0.2</mu1>
-      <mu2>0.2</mu2>
-    </gazebo>
-    <gazebo reference="wheel_fl">
-        <mu1>10.0</mu1>
-        <mu2>10.0</mu2>
-        <kp>100000.0</kp>
-        <kd>10.0</kd>
-        <minDepth>0.001</minDepth>
-        <maxVel>0.1</maxVel>
-        <fdir1>1 1 0</fdir1>
-    </gazebo>
-    <gazebo reference="wheel_fr">
-        <mu1>10.0</mu1>
-        <mu2>10.0</mu2>
-        <kp>100000.0</kp>
-        <kd>10.0</kd>
-        <minDepth>0.001</minDepth>
-        <maxVel>0.1</maxVel>
-        <fdir1>1 -1 0</fdir1>
-    </gazebo>
-    <gazebo reference="wheel_bl">
-        <mu1>10.0</mu1>
-        <mu2>10.0</mu2>
-        <kp>100000.0</kp>
-        <kd>10.0</kd>
-        <minDepth>0.001</minDepth>
-        <maxVel>0.1</maxVel>
-        <fdir1>1 -1 0</fdir1>
-    </gazebo>
-    <gazebo reference="wheel_br">
-        <mu1>10.0</mu1>
-        <mu2>10.0</mu2>
-        <kp>100000.0</kp>
-        <kd>10.0</kd>
-        <minDepth>0.001</minDepth>
-        <maxVel>0.1</maxVel>
-        <fdir1>1 1 0</fdir1>
-    </gazebo>
-    <!-- Joint State Publisher -->
-    <!-- <gazebo>
-      <plugin filename="libignition-gazebo6-joint-state-publisher-system.so" name="ignition::gazebo::systems::JointStatePublisher">
-      </plugin>
-    </gazebo> -->
-    <!-- Mecanum Drive Plugin - Handles all wheels and kinematics! -->
     <gazebo>
-      <plugin filename="libignition-gazebo6-mecanum-drive-system.so" name="ignition::gazebo::systems::MecanumDrive">
-        <front_left_joint>wheel_fl_joint</front_left_joint>
-        <front_right_joint>wheel_fr_joint</front_right_joint>
-        <back_left_joint>wheel_bl_joint</back_left_joint>
-        <back_right_joint>wheel_br_joint</back_right_joint>
-        <wheel_separation>0.4</wheel_separation>
-        <wheel_diameter>0.2</wheel_diameter>
-        <max_linear_speed>5.0</max_linear_speed>
-        <max_angular_speed>5.0</max_angular_speed>
-        <topic>${robot_ns}/cmd_vel</topic>
-      </plugin>
-    </gazebo>
-    <gazebo>
-      <plugin filename="libignition-gazebo6-joint-controller-system.so" name="ignition::gazebo::systems::JointController">
+        <plugin
+        filename="ignition-gazebo-velocity-control-system"
+        name="gz::sim::systems::VelocityControl">
+        </plugin>
+        <plugin filename="ignition-gazebo-joint-state-publisher-system"
+        name="ignition::gazebo::systems::JointStatePublisher">
+        </plugin>
+        <!-- ign topic -t "/model/{bot_name}/joint/arm_base/cmd_vel" -m ignition.msgs.Double -p "data: 10.0" -->
+        <plugin filename="ignition-gazebo-joint-controller-system"
+        name="gz::sim::systems::JointController">
         <joint_name>arm_joint_1</joint_name>
-        <topic>/${robot_ns}/cmd_shoulder</topic>
-      </plugin>
-    </gazebo>
-    <gazebo>
-      <plugin filename="libignition-gazebo6-joint-controller-system.so" name="ignition::gazebo::systems::JointController">
+        </plugin>
+        <plugin filename="ignition-gazebo-joint-controller-system"
+        name="gz::sim::systems::JointController">
         <joint_name>arm_joint_2</joint_name>
-        <topic>/${robot_ns}/cmd_elbow</topic>
-      </plugin>
-    </gazebo>
-    <gazebo>
-      <plugin filename="libignition-gazebo6-joint-state-publisher-system.so" name="ignition::gazebo::systems::JointStatePublisher">
-        <joint_name>arm_joint_1</joint_name>
-        <joint_name>arm_joint_2</joint_name>
-      </plugin>
-    </gazebo>
-    <gazebo>
-      <plugin filename="libignition-gazebo6-odometry-publisher-system.so" name="ignition::gazebo::systems::OdometryPublisher">
-        <body_name>base_link</body_name>
-        <odom_publish_frequency>100</odom_publish_frequency>
-        <odom_topic>${robot_ns}/odom</odom_topic>
-        <tf_topic>${robot_ns}/tf</tf_topic>
-      </plugin>
-    </gazebo>
-    <gazebo reference="arm_base_link"/>
-    <gazebo reference="arm_joint_1"/>
-    <gazebo reference="arm_joint_2"/>
-    <gazebo reference="arm_joint_1">
-      <implicitSpringDamper>true</implicitSpringDamper>
-    </gazebo>
-    <gazebo reference="arm_joint_2">
-      <implicitSpringDamper>true</implicitSpringDamper>
+        </plugin>
+        <plugin filename="libignition-gazebo6-odometry-publisher-system.so"
+        name="ignition::gazebo::systems::OdometryPublisher">
+          <body_name>base_link</body_name>
+          <odom_publish_frequency>100</odom_publish_frequency>
+          <odom_topic>${robot_ns}/odom</odom_topic>
+          <tf_topic>${robot_ns}/tf</tf_topic>
+        </plugin>
     </gazebo>
   </xacro:macro>

File: sr_description/urdf/runner_gazebo.urdf.xacro (robot description, xacro)
@@ -2,84 +2,24 @@
 <robot xmlns:xacro="http://www.ros.org/wiki/xacro">
   <xacro:macro name="gazebo_setup_run" params="robot_ns">
-    <gazebo reference="base_link">
-      <mu1>0.2</mu1>
-      <mu2>0.2</mu2>
-    </gazebo>
-    <gazebo reference="wheel_fl">
-        <mu1>10.0</mu1>
-        <mu2>10.0</mu2>
-        <kp>100000.0</kp>
-        <kd>10.0</kd>
-        <minDepth>0.001</minDepth>
-        <maxVel>0.1</maxVel>
-        <fdir1>1 1 0</fdir1>
-    </gazebo>
-    <gazebo reference="wheel_fr">
-        <mu1>10.0</mu1>
-        <mu2>10.0</mu2>
-        <kp>100000.0</kp>
-        <kd>10.0</kd>
-        <minDepth>0.001</minDepth>
-        <maxVel>0.1</maxVel>
-        <fdir1>1 -1 0</fdir1>
-    </gazebo>
-    <gazebo reference="wheel_bl">
-        <mu1>10.0</mu1>
-        <mu2>10.0</mu2>
-        <kp>100000.0</kp>
-        <kd>10.0</kd>
-        <minDepth>0.001</minDepth>
-        <maxVel>0.1</maxVel>
-        <fdir1>1 -1 0</fdir1>
-    </gazebo>
-    <gazebo reference="wheel_br">
-        <mu1>10.0</mu1>
-        <mu2>10.0</mu2>
-        <kp>100000.0</kp>
-        <kd>10.0</kd>
-        <minDepth>0.001</minDepth>
-        <maxVel>0.1</maxVel>
-        <fdir1>1 1 0</fdir1>
-    </gazebo>
-    <!-- Joint State Publisher -->
     <gazebo>
-      <plugin filename="libignition-gazebo6-joint-state-publisher-system.so" name="ignition::gazebo::systems::JointStatePublisher">
-      </plugin>
-    </gazebo>
-    <!-- Mecanum Drive Plugin - Handles all wheels and kinematics! -->
-    <gazebo>
-      <plugin filename="libignition-gazebo6-mecanum-drive-system.so" name="ignition::gazebo::systems::MecanumDrive">
-        <front_left_joint>wheel_fl_joint</front_left_joint>
-        <front_right_joint>wheel_fr_joint</front_right_joint>
-        <back_left_joint>wheel_bl_joint</back_left_joint>
-        <back_right_joint>wheel_br_joint</back_right_joint>
-        <wheel_separation>0.4</wheel_separation>
-        <wheel_diameter>0.2</wheel_diameter>
-        <max_linear_speed>5.0</max_linear_speed>
-        <max_angular_speed>5.0</max_angular_speed>
-        <topic>${robot_ns}/cmd_vel</topic>
-      </plugin>
-    </gazebo>
-    <gazebo>
-      <plugin filename="libignition-gazebo6-joint-controller-system.so" name="ignition::gazebo::systems::JointController">
+        <plugin
+        filename="ignition-gazebo-velocity-control-system"
+        name="gz::sim::systems::VelocityControl">
+        </plugin>
+        <plugin filename="ignition-gazebo-joint-state-publisher-system"
+        name="ignition::gazebo::systems::JointStatePublisher">
+        </plugin>
+        <!-- ign topic -t "/model/{bot_name}/joint/arm_base/cmd_vel" -m ignition.msgs.Double -p "data: 10.0" -->
+        <plugin filename="ignition-gazebo-joint-controller-system"
+        name="gz::sim::systems::JointController">
         <joint_name>piston_rod_joint</joint_name>
-        <topic>/${robot_ns}/cmd_piston</topic>
-      </plugin>
-    </gazebo>
-    <gazebo>
-      <plugin filename="libignition-gazebo6-odometry-publisher-system.so" name="ignition::gazebo::systems::OdometryPublisher">
-        <body_name>base_link</body_name>
-        <odom_publish_frequency>100</odom_publish_frequency>
-        <odom_topic>${robot_ns}/odom</odom_topic>
-        <tf_topic>${robot_ns}/tf</tf_topic>
-      </plugin>
-    </gazebo>
-    <!-- ================= ACTUATOR LINKS ================= -->
-    <gazebo reference="piston_base"/>
-    <gazebo reference="piston_rod"/>
-    <gazebo reference="piston_head"/>
-    <!-- ================= ARM JOINT DYNAMICS ================= -->
-    <gazebo reference="piston_rod_joint">
-      <implicitSpringDamper>true</implicitSpringDamper>
+        </plugin>
+        <plugin filename="libignition-gazebo6-odometry-publisher-system.so"
+        name="ignition::gazebo::systems::OdometryPublisher">
+          <body_name>base_link</body_name>
+          <odom_publish_frequency>100</odom_publish_frequency>
+          <odom_topic>${robot_ns}/odom</odom_topic>
+          <tf_topic>${robot_ns}/tf</tf_topic>
+        </plugin>
     </gazebo>
   </xacro:macro>

File: sr_description/urdf/wheel.urdf.xacro (robot description, xacro)
@@ -30,5 +30,5 @@
       <axis xyz="0 1 0"/>
       <limit effort="100.0" velocity="40.0" lower="-3.14159" upper="3.14159"/>
-      <dynamics damping="0.1" friction="0.1"/>
+      <dynamics damping="0.05" friction="0.1"/>
     </joint>
     <!-- ================= FRONT RIGHT WHEEL ================= -->
@@ -60,5 +60,5 @@
       <axis xyz="0 1 0"/>
       <limit effort="100.0" velocity="40.0" lower="-3.14159" upper="3.14159"/>
-      <dynamics damping="0.1" friction="0.1"/>
+      <dynamics damping="0.05" friction="0.1"/>
     </joint>
     <!-- ================= REAR LEFT WHEEL ================= -->
@@ -90,5 +90,5 @@
       <axis xyz="0 1 0"/>
       <limit effort="100.0" velocity="40.0" lower="-3.14159" upper="3.14159"/>
-      <dynamics damping="0.1" friction="0.1"/>
+      <dynamics damping="0.05" friction="0.1"/>
     </joint>
     <!-- ================= REAR RIGHT WHEEL ================= -->
@@ -120,5 +120,5 @@
       <axis xyz="0 1 0"/>
       <limit effort="100.0" velocity="40.0" lower="-3.14159" upper="3.14159"/>
-      <dynamics damping="0.1" friction="0.1"/>
+      <dynamics damping="0.05" friction="0.1"/>
     </joint>
   </xacro:macro>

Commit message: debugging-3

File: sr_description/urdf/arm.urdf.xacro (robot description, xacro)
@@ -22,10 +22,10 @@
       </visual>
       <!-- Collision (simple box for stability) -->
-      <!-- <collision>
+      <collision>
         <origin xyz="0 0 0.1" rpy="0 0 0"/>
         <geometry>
           <box size="0.05 0.05 0.15" scale="5 5 3"/>
         </geometry>
-      </collision> -->
+      </collision>
     </link>
     <!-- ARM LINK 2 -->
@@ -49,10 +49,10 @@
       </visual>
       <!-- Collision -->
-      <!-- <collision>
+      <collision>
         <origin xyz="0 0 0.1" rpy="0 0 0"/>
         <geometry>
           <box size="0.04 0.04 0.10" scale="5 5 2"/>
         </geometry>
-      </collision> -->
+      </collision>
     </link>
     <!-- JOINT 1 -->

File: sr_description/urdf/base.urdf.xacro (robot description, xacro)
@@ -21,5 +21,5 @@
       <inertial>
         <origin xyz="0 0 0"/>
-        <mass value="1.0"/>
+        <mass value="3.0"/>
         <inertia ixx="0.1" iyy="0.1" izz="0.1"
                 ixy="0" ixz="0" iyz="0"/>

File: sr_description/urdf/lifter_gazebo.urdf.xacro (robot description, xacro)
@@ -4,4 +4,28 @@
     <gazebo>
         <static>false</static>
+    </gazebo>
+    <gazebo reference="wheel_fl_link">
+      <mu1>0.8</mu1>
+      <mu2>0.8</mu2>
+      <kp>1000000.0</kp>
+      <kd>100.0</kd>
+    </gazebo>
+    <gazebo reference="wheel_fr_link">
+      <mu1>0.8</mu1>
+      <mu2>0.8</mu2>
+      <kp>1000000.0</kp>
+      <kd>100.0</kd>
+    </gazebo>
+    <gazebo reference="wheel_bl_link">
+      <mu1>0.8</mu1>
+      <mu2>0.8</mu2>
+      <kp>1000000.0</kp>
+      <kd>100.0</kd>
+    </gazebo>
+    <gazebo reference="wheel_br_link">
+      <mu1>0.8</mu1>
+      <mu2>0.8</mu2>
+      <kp>1000000.0</kp>
+      <kd>100.0</kd>
     </gazebo>
     <gazebo>

File: sr_description/urdf/runner_gazebo.urdf.xacro (robot description, xacro)
@@ -4,4 +4,28 @@
     <gazebo>
         <static>false</static>
+    </gazebo>
+    <gazebo reference="wheel_fl_link">
+      <mu1>0.8</mu1>
+      <mu2>0.8</mu2>
+      <kp>1000000.0</kp>
+      <kd>100.0</kd>
+    </gazebo>
+    <gazebo reference="wheel_fr_link">
+      <mu1>0.8</mu1>
+      <mu2>0.8</mu2>
+      <kp>1000000.0</kp>
+      <kd>100.0</kd>
+    </gazebo>
+    <gazebo reference="wheel_bl_link">
+      <mu1>0.8</mu1>
+      <mu2>0.8</mu2>
+      <kp>1000000.0</kp>
+      <kd>100.0</kd>
+    </gazebo>
+    <gazebo reference="wheel_br_link">
+      <mu1>0.8</mu1>
+      <mu2>0.8</mu2>
+      <kp>1000000.0</kp>
+      <kd>100.0</kd>
     </gazebo>
     <gazebo>

Commit message: urdf draft-4

File: sr_description/urdf/arm.urdf.xacro (robot description, xacro)
@@ -57,5 +57,5 @@
     </link>
     <!-- JOINT 1 -->
-    <joint name="arm_joint_1" type="revolute">
+    <joint name="arm_joint_1" type="fixed">
       <parent link="arm_base_link"/>
       <child link="arm_link_1"/>
@@ -66,5 +66,5 @@
     </joint>
     <!-- JOINT 2 -->
-    <joint name="arm_joint_2" type="revolute">
+    <joint name="arm_joint_2" type="fixed">
       <parent link="arm_link_1"/>
       <child link="arm_link_2"/>

File: sr_description/urdf/wheel.urdf.xacro (robot description, xacro)
@@ -21,14 +21,14 @@
         <origin xyz="0 0 0"/>
         <mass value="0.5"/>
-        <inertia ixx="0.001" iyy="0.001" izz="0.001" ixy="0" ixz="0" iyz="0"/>
+        <inertia ixx="0.000417" iyy="0.0005" izz="0.000417" ixy="0" ixz="0" iyz="0"/>
       </inertial>
     </link>
     <!-- Front Left Joint -->
-    <joint name="wheel_fl_joint" type="revolute">
+    <joint name="wheel_fl_joint" type="continuous">
       <parent link="base_link"/>
       <child link="wheel_fl_link"/>
       <origin xyz="0.20 0.20 0.0" rpy="0 0 0"/>
       <axis xyz="0 1 0"/>
-      <limit effort="100.0" velocity="40.0" lower="-3.14159" upper="3.14159"/>
+      <limit effort="100.0" velocity="40.0" lower="-100.0" upper="100.0"/>
       <dynamics damping="0.05" friction="0.1"/>
     </joint>
@@ -52,14 +52,14 @@
         <origin xyz="0 0 0"/>
         <mass value="0.5"/>
-        <inertia ixx="0.001" iyy="0.001" izz="0.001" ixy="0" ixz="0" iyz="0"/>
+        <inertia ixx="0.000417" iyy="0.0005" izz="0.000417" ixy="0" ixz="0" iyz="0"/>
       </inertial>
     </link>
     <!-- Front Right Joint -->
-    <joint name="wheel_fr_joint" type="revolute">
+    <joint name="wheel_fr_joint" type="continuous">
       <parent link="base_link"/>
       <child link="wheel_fr_link"/>
       <origin xyz="0.20 -0.20 0.0" rpy="0 0 0"/>
       <axis xyz="0 1 0"/>
-      <limit effort="100.0" velocity="40.0" lower="-3.14159" upper="3.14159"/>
+      <limit effort="100.0" velocity="40.0" lower="-100.0" upper="100.0"/>
       <dynamics damping="0.05" friction="0.1"/>
     </joint>
@@ -83,14 +83,14 @@
         <origin xyz="0 0 0"/>
         <mass value="0.5"/>
-        <inertia ixx="0.001" iyy="0.001" izz="0.001" ixy="0" ixz="0" iyz="0"/>
+        <inertia ixx="0.000417" iyy="0.0005" izz="0.000417" ixy="0" ixz="0" iyz="0"/>
       </inertial>
     </link>
     <!-- Rear Left Joint -->
-    <joint name="wheel_bl_joint" type="revolute">
+    <joint name="wheel_bl_joint" type="continuous">
       <parent link="base_link"/>
       <child link="wheel_bl_link"/>
       <origin xyz="-0.20 0.20 0.0" rpy="0 0 0"/>
       <axis xyz="0 1 0"/>
-      <limit effort="100.0" velocity="40.0" lower="-3.14159" upper="3.14159"/>
+      <limit effort="100.0" velocity="40.0" lower="-100.0" upper="100.0"/>
       <dynamics damping="0.05" friction="0.1"/>
     </joint>
@@ -114,14 +114,14 @@
         <origin xyz="0 0 0"/>
         <mass value="0.5"/>
-        <inertia ixx="0.001" iyy="0.001" izz="0.001" ixy="0" ixz="0" iyz="0"/>
+        <inertia ixx="0.000417" iyy="0.0005" izz="0.000417" ixy="0" ixz="0" iyz="0"/>
       </inertial>
     </link>
     <!-- Rear Right Joint -->
-    <joint name="wheel_br_joint" type="revolute">
+    <joint name="wheel_br_joint" type="continuous">
       <parent link="base_link"/>
       <child link="wheel_br_link"/>
       <origin xyz="-0.20 -0.20 0.0" rpy="0 0 0"/>
       <axis xyz="0 1 0"/>
-      <limit effort="100.0" velocity="40.0" lower="-3.14159" upper="3.14159"/>
+      <limit effort="100.0" velocity="40.0" lower="-100.0" upper="100.0"/>
       <dynamics damping="0.05" friction="0.1"/>
     </joint>

Commit message: debugging-4

File: sr_description/urdf/arm.urdf.xacro (robot description, xacro)
@@ -57,5 +57,5 @@
     </link>
     <!-- JOINT 1 -->
-    <joint name="arm_joint_1" type="fixed">
+    <joint name="arm_joint_1" type="revolute">
       <parent link="arm_base_link"/>
       <child link="arm_link_1"/>
@@ -63,14 +63,14 @@
       <axis xyz="0 1 0"/>
       <limit effort="100.0" velocity="10.0" lower="0.0" upper="1.5708"/>
-      <dynamics damping="0.1" friction="0.1"/>
+      <dynamics damping="2.0" friction="0.1"/>
     </joint>
     <!-- JOINT 2 -->
-    <joint name="arm_joint_2" type="fixed">
+    <joint name="arm_joint_2" type="revolute">
       <parent link="arm_link_1"/>
       <child link="arm_link_2"/>
-      <origin xyz="0 0 0.155" rpy="0 0 0"/>
+      <origin xyz="0 0 0.115" rpy="0 0 0"/>
       <axis xyz="0 1 0"/>
       <limit effort="100.0" velocity="10.0" lower="0.0" upper="1.5708"/>
-      <dynamics damping="0.1" friction="0.1"/>
+      <dynamics damping="2.0" friction="0.1"/>
     </joint>
   </xacro:macro>

File: sr_description/urdf/wheel.urdf.xacro (robot description, xacro)
@@ -30,5 +30,5 @@
       <origin xyz="0.20 0.20 0.0" rpy="0 0 0"/>
       <axis xyz="0 1 0"/>
-      <limit effort="100.0" velocity="40.0" lower="-100.0" upper="100.0"/>
+      <limit effort="100.0" velocity="40.0" lower="-1000.0" upper="1000.0"/>
       <dynamics damping="0.05" friction="0.1"/>
     </joint>
@@ -61,5 +61,5 @@
       <origin xyz="0.20 -0.20 0.0" rpy="0 0 0"/>
       <axis xyz="0 1 0"/>
-      <limit effort="100.0" velocity="40.0" lower="-100.0" upper="100.0"/>
+      <limit effort="100.0" velocity="40.0" lower="-1000.0" upper="1000.0"/>
       <dynamics damping="0.05" friction="0.1"/>
     </joint>
@@ -92,5 +92,5 @@
       <origin xyz="-0.20 0.20 0.0" rpy="0 0 0"/>
       <axis xyz="0 1 0"/>
-      <limit effort="100.0" velocity="40.0" lower="-100.0" upper="100.0"/>
+      <limit effort="100.0" velocity="40.0" lower="-1000.0" upper="1000.0"/>
       <dynamics damping="0.05" friction="0.1"/>
     </joint>
@@ -123,5 +123,5 @@
       <origin xyz="-0.20 -0.20 0.0" rpy="0 0 0"/>
       <axis xyz="0 1 0"/>
-      <limit effort="100.0" velocity="40.0" lower="-100.0" upper="100.0"/>
+      <limit effort="100.0" velocity="40.0" lower="-1000.0" upper="1000.0"/>
       <dynamics damping="0.05" friction="0.1"/>
     </joint>
