Commit message: urdf draft -5

File: sr_description/urdf/arm.urdf.xacro (robot description, xacro)
@@ -7,9 +7,9 @@
       <inertial>
         <origin xyz="0 0 0.1" rpy="0 0 0"/>
-        <mass value="0.5"/>
+        <mass value="0.25"/>
         <inertia
-          ixx="0.01" ixy="0.0" ixz="0.0"
-          iyy="0.01" iyz="0.0"
-          izz="0.01"/>
+          ixx="0.00052083" ixy="0.0" ixz="0.0"
+          iyy="0.00052083" iyz="0.0"
+          izz="0.00010417"/>
       </inertial>
       <!-- Visual -->
@@ -34,9 +34,9 @@
       <inertial>
         <origin xyz="0 0 0.1" rpy="0 0 0"/>
-        <mass value="0.35"/>
+        <mass value="0.12"/>
         <inertia
-          ixx="0.005" ixy="0.0" ixz="0.0"
-          iyy="0.005" iyz="0.0"
-          izz="0.005"/>
+          ixx="0.000116" ixy="0.0" ixz="0.0"
+          iyy="0.000116" iyz="0.0"
+          izz="0.000032"/>
       </inertial>
       <!-- Visual -->

File: sr_description/urdf/lifter_gazebo.urdf.xacro (robot description, xacro)
@@ -49,4 +49,17 @@
           <cmd_vel_topic>/model/lifter1/joint/wheel_br_joint/cmd_vel</cmd_vel_topic>
       </plugin>
+      <plugin filename="libignition-gazebo-joint-controller-system.so"
+              name="ignition::gazebo::systems::JointController">
+          <joint_name>arm_joint_1</joint_name>
+          <cmd_vel_topic>/model/lifter1/joint/arm_joint_1/cmd_vel</cmd_vel_topic>
+      </plugin>
+      <plugin filename="libignition-gazebo-joint-controller-system.so"
+              name="ignition::gazebo::systems::JointController">
+          <joint_name>arm_joint_2</joint_name>
+          <cmd_vel_topic>/model/lifter1/joint/arm_joint_2/cmd_vel</cmd_vel_topic>
+      </plugin>
+      <plugin filename="libignition-gazebo-link-attacher-system.so"
+        name="ignition::gazebo::systems::LinkAttacher">
+      </plugin>
       <plugin filename="libignition-gazebo-odometry-publisher-system.so" name="ignition::gazebo::systems::OdometryPublisher">
           <odom_topic>/lifter1/odom</odom_topic>

File: sr_description/urdf/runner_gazebo.urdf.xacro (robot description, xacro)
@@ -49,4 +49,12 @@
           <topic>/model/runner1/joint/wheel_br_joint/cmd_vel</topic>
       </plugin>
+      <plugin filename="libignition-gazebo-link-attacher-system.so"
+        name="ignition::gazebo::systems::LinkAttacher">
+      </plugin>
+      <plugin filename="libignition-gazebo-joint-controller-system.so"
+              name="ignition::gazebo::systems::JointController">
+          <joint_name>piston_rod_joint</joint_name>
+          <cmd_vel_topic>/model/runner1/joint/piston_rod_joint/cmd_vel</cmd_vel_topic>
+      </plugin>
       <plugin filename="libignition-gazebo-odometry-publisher-system.so" name="ignition::gazebo::systems::OdometryPublisher">
           <odom_topic>/runner1/odom</odom_topic>

Commit message: urdf draft-6

File: sr_description/urdf/arm.urdf.xacro (robot description, xacro)
@@ -2,59 +2,5 @@
 <robot xmlns:xacro="http://www.ros.org/wiki/xacro">
   <xacro:macro name="create_arm">
-    <!-- ARM LINK 1 -->
-    <link name="arm_link_1">
-      <!-- Inertia -->
-      <inertial>
-        <origin xyz="0 0 0.1" rpy="0 0 0"/>
-        <mass value="0.25"/>
-        <inertia
-          ixx="0.00052083" ixy="0.0" ixz="0.0"
-          iyy="0.00052083" iyz="0.0"
-          izz="0.00010417"/>
-      </inertial>
-      <!-- Visual -->
-      <visual>
-        <origin xyz="0 0 0" rpy="0 0 0"/>
-        <geometry>
-          <mesh filename="package://sr_description/meshes/arm_link.dae"
-                scale="5 5 3"/>
-        </geometry>
-      </visual>
-      <!-- Collision (simple box for stability) -->
-      <collision>
-        <origin xyz="0 0 0.1" rpy="0 0 0"/>
-        <geometry>
-          <box size="0.05 0.05 0.15" scale="5 5 3"/>
-        </geometry>
-      </collision>
-    </link>
-    <!-- ARM LINK 2 -->
-    <link name="arm_link_2">
-      <!-- Inertia -->
-      <inertial>
-        <origin xyz="0 0 0.1" rpy="0 0 0"/>
-        <mass value="0.12"/>
-        <inertia
-          ixx="0.000116" ixy="0.0" ixz="0.0"
-          iyy="0.000116" iyz="0.0"
-          izz="0.000032"/>
-      </inertial>
-      <!-- Visual -->
-      <visual>
-        <origin xyz="0 0 0" rpy="0 0 0"/>
-        <geometry>
-          <mesh filename="package://sr_description/meshes/arm_elbow.dae"
-                scale="5 5 2"/>
-        </geometry>
-      </visual>
-      <!-- Collision -->
-      <collision>
-        <origin xyz="0 0 0.1" rpy="0 0 0"/>
-        <geometry>
-          <box size="0.04 0.04 0.10" scale="5 5 2"/>
-        </geometry>
-      </collision>
-    </link>
-    <!-- JOINT 1 -->
+    <!-- Joint 1: Base to Arm Link 1 -->
     <joint name="arm_joint_1" type="revolute">
       <parent link="arm_base_link"/>
@@ -62,16 +8,71 @@
       <origin xyz="0 0 0" rpy="0 0 0"/>
       <axis xyz="0 1 0"/>
-      <limit effort="100.0" velocity="10.0" lower="0.0" upper="1.5708"/>
-      <dynamics damping="2.0" friction="0.1"/>
+      <limit effort="50.0" velocity="2.0" lower="0.0" upper="1.5708"/>
+      <dynamics damping="0.5" friction="0.1"/>
     </joint>
-    <!-- JOINT 2 -->
+    <!-- ================= ARM LINK 1 ================= -->
+    <link name="arm_link_1">
+      <visual>
+        <origin xyz="0 0 0.125" rpy="0 0 0"/>
+        <geometry>
+          <cylinder radius="0.035" length="0.25"/>
+        </geometry>
+        <material name="dark_grey"/>
+      </visual>
+      <collision>
+        <origin xyz="0 0 0.125" rpy="0 0 0"/>
+        <geometry>
+          <cylinder radius="0.035" length="0.25"/>
+        </geometry>
+      </collision>
+      <inertial>
+        <origin xyz="0 0 0.125"/>
+        <mass value="0.25"/>
+        <inertia ixx="0.001458" iyy="0.001458" izz="0.0003125" ixy="0" ixz="0" iyz="0"/>
+      </inertial>
+    </link>
+    <!-- Joint 2: Arm Link 1 to Arm Link 2 -->
     <joint name="arm_joint_2" type="revolute">
       <parent link="arm_link_1"/>
       <child link="arm_link_2"/>
-      <origin xyz="0 0 0.115" rpy="0 0 0"/>
+      <origin xyz="0 0 0.25" rpy="0 0 0"/>
       <axis xyz="0 1 0"/>
-      <limit effort="100.0" velocity="10.0" lower="0.0" upper="1.5708"/>
-      <dynamics damping="2.0" friction="0.1"/>
+      <limit effort="50.0" velocity="2.0" lower="0.0" upper="1.5708"/>
+      <dynamics damping="0.5" friction="0.1"/>
     </joint>
+    <!-- ================= ARM LINK 2 (GRABBER) ================= -->
+    <link name="arm_link_2">
+      <visual>
+        <origin xyz="0 0 0.06" rpy="0 0 0"/>
+        <geometry>
+          <cylinder radius="0.035" length="0.12"/>
+        </geometry>
+        <material name="dark_grey"/>
+      </visual>
+      <collision>
+        <origin xyz="0 0 0.06" rpy="0 0 0"/>
+        <geometry>
+          <cylinder radius="0.035" length="0.12"/>
+        </geometry>
+      </collision>
+      <inertial>
+        <origin xyz="0 0 0.06"/>
+        <mass value="0.1"/>
+        <inertia ixx="0.0001825" iyy="0.0001825" izz="0.000125" ixy="0" ixz="0" iyz="0"/>
+      </inertial>
+    </link>
+    <joint name="gripper_joint" type="fixed">
+      <parent link="arm_link_2"/>
+      <child link="gripper_link"/>
+      <origin xyz="0 0 0.12" rpy="0 0 0"/>
+    </joint>
+    <!-- ================= GRIPPER LINK (EMPTY - FOR GRABBING) ================= -->
+    <link name="gripper_link">
+      <inertial>
+        <origin xyz="0 0 0"/>
+        <mass value="0.01"/>
+        <inertia ixx="0.00001" iyy="0.00001" izz="0.00001" ixy="0" ixz="0" iyz="0"/>
+      </inertial>
+    </link>
   </xacro:macro>
 </robot>

Commit message: debugging -6

File: sr_description/urdf/arm.urdf.xacro (robot description, xacro)
@@ -69,4 +69,16 @@
     <!-- ================= GRIPPER LINK (EMPTY - FOR GRABBING) ================= -->
     <link name="gripper_link">
+      <visual>
+          <origin xyz="0 0 0.01" rpy="0 0 0"/>
+          <geometry>
+            <cylinder radius="0.035" length="0.02"/>
+          </geometry>
+      </visual>
+      <collision>
+        <origin xyz="0 0 0.01" rpy="0 0 0"/>
+        <geometry>
+          <cylinder radius="0.035" length="0.02"/>
+        </geometry>
+      </collision>
       <inertial>
         <origin xyz="0 0 0"/>

Commit message: control draft-6

File: sr_description/urdf/arm.urdf.xacro (robot description, xacro)
@@ -62,8 +62,11 @@
       </inertial>
     </link>
-    <joint name="gripper_joint" type="fixed">
+    <joint name="gripper_joint" type="revolute">
       <parent link="arm_link_2"/>
       <child link="gripper_link"/>
       <origin xyz="0 0 0.12" rpy="0 0 0"/>
+      <axis xyz="0 0 1"/>
+      <limit effort="1.0" velocity="0.01" lower="0" upper="0"/>
+      <dynamics damping="0.0" friction="0.0"/>
     </joint>
     <!-- ================= GRIPPER LINK (EMPTY - FOR GRABBING) ================= -->

Commit message: debugging-7

File: sr_description/urdf/arm.urdf.xacro (robot description, xacro)
@@ -6,5 +6,5 @@
       <parent link="arm_base_link"/>
       <child link="arm_link_1"/>
-      <origin xyz="0 0 0" rpy="0 0 0"/>
+      <origin xyz="0 0 0.15" rpy="0 0 0"/>
       <axis xyz="0 1 0"/>
       <limit effort="50.0" velocity="2.0" lower="0.0" upper="1.5708"/>
@@ -85,5 +85,5 @@
       </collision>
       <inertial>
-        <origin xyz="0 0 0"/>
+        <origin xyz="0 0 0.01"/>
         <mass value="0.01"/>
         <inertia ixx="0.00001" iyy="0.00001" izz="0.00001" ixy="0" ixz="0" iyz="0"/>

File: sr_description/urdf/lifter_gazebo.urdf.xacro (robot description, xacro)
@@ -60,4 +60,6 @@
       </plugin>
       <plugin filename="libignition_link_attacher.so" name="ignition_link_attacher">
+          <attach_distance>0.15</attach_distance>
+          <detach_distance>0.2</detach_distance>
       </plugin>
       <plugin filename="libignition-gazebo-odometry-publisher-system.so" name="ignition::gazebo::systems::OdometryPublisher">

Commit message: debugging -8

File: sr_description/urdf/arm.urdf.xacro (robot description, xacro)
@@ -65,5 +65,5 @@
       <parent link="arm_link_2"/>
       <child link="gripper_link"/>
-      <origin xyz="0 0 0.12" rpy="0 0 0"/>
+      <origin xyz="0 0 0.11" rpy="0 0 0"/>
       <axis xyz="0 0 1"/>
       <limit effort="1.0" velocity="0.01" lower="0" upper="0"/>

File: sr_description/urdf/lifter_gazebo.urdf.xacro (robot description, xacro)
@@ -60,6 +60,4 @@
       </plugin>
       <plugin filename="libignition_link_attacher.so" name="ignition_link_attacher">
-          <attach_distance>0.15</attach_distance>
-          <detach_distance>0.2</detach_distance>
       </plugin>
       <plugin filename="libignition-gazebo-odometry-publisher-system.so" name="ignition::gazebo::systems::OdometryPublisher">

Commit message: debugging - 9

File: sr_description/urdf/arm.urdf.xacro (robot description, xacro)
@@ -68,5 +68,5 @@
       <axis xyz="0 0 1"/>
       <limit effort="1.0" velocity="0.01" lower="0" upper="0"/>
-      <dynamics damping="0.0" friction="0.0"/>
+      <dynamics damping="0.1" friction="0.1"/>
     </joint>
     <!-- ================= GRIPPER LINK (EMPTY - FOR GRABBING) ================= -->

Commit message: complete draft -4

File: sr_description/urdf/arm.urdf.xacro (robot description, xacro)
@@ -68,5 +68,5 @@
       <axis xyz="0 0 1"/>
       <limit effort="1.0" velocity="0.01" lower="0" upper="0"/>
-      <dynamics damping="0.1" friction="0.1"/>
+      <dynamics damping="100.0" friction="100.0"/>
     </joint>
     <!-- ================= GRIPPER LINK (EMPTY - FOR GRABBING) ================= -->

File: sr_description/urdf/lifter_gazebo.urdf.xacro (robot description, xacro)
@@ -28,4 +28,7 @@
       <kp>1000000.0</kp>
       <kd>100.0</kd>
+    </gazebo>
+    <gazebo reference="gripper_joint">
+        <preserveFixedJoint>true</preserveFixedJoint>
     </gazebo>
     <gazebo>

Commit message: debugging-11

File: sr_description/urdf/arm.urdf.xacro (robot description, xacro)
@@ -62,8 +62,8 @@
       </inertial>
     </link>
-    <joint name="gripper_joint" type="revolute">
+    <joint name="gripper_joint" type="fixed">
       <parent link="arm_link_2"/>
       <child link="gripper_link"/>
-      <origin xyz="0 0 0.11" rpy="0 0 0"/>
+      <origin xyz="0 0 0.14" rpy="0 0 0"/>
       <axis xyz="0 0 1"/>
       <limit effort="1.0" velocity="0.01" lower="0" upper="0"/>
@@ -73,5 +73,5 @@
     <link name="gripper_link">
       <visual>
-          <origin xyz="0 0 0.01" rpy="0 0 0"/>
+          <origin xyz="0 0 -0.01" rpy="0 0 0"/>
           <geometry>
             <cylinder radius="0.035" length="0.02"/>
@@ -79,5 +79,5 @@
       </visual>
       <collision>
-        <origin xyz="0 0 0.01" rpy="0 0 0"/>
+        <origin xyz="0 0 -0.01" rpy="0 0 0"/>
         <geometry>
           <cylinder radius="0.035" length="0.02"/>
@@ -85,5 +85,5 @@
       </collision>
       <inertial>
-        <origin xyz="0 0 0.01"/>
+        <origin xyz="0 0 -0.01"/>
         <mass value="0.01"/>
         <inertia ixx="0.00001" iyy="0.00001" izz="0.00001" ixy="0" ixz="0" iyz="0"/>
